File: EP91Starlet.kicad_sch (KiCad schematic)
At the start: 4 parts, among them M1 Module-mega-mcu64-0.1, M2 Module-wbo-0.5, M3 Module-vr-max9924-0.1, M4 Module-knock-0.2

Commit message: more testing
Connections:
- net GND: now reaches M4.E2 (GND)
- net GND: now also M1.G (GND), M2.G (GND), M3.G (GND)
- net at M4.W2 (VREF): now also M1.N22 (V33)
- net at M1.S26 (IN_ADC10/EINT0_(VR_CRK)): now also M3.E3 (OUT)
- net at M1.W12 (CAN1H): now also M2.W3 (CANL)
- net at M1.W13 (CAN1L): now also M2.W4 (CANH)
Other:
- moved on the sheet: M3
Changed lines of the file:
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@@
 (kicad_sch (version 20230121) (generator eeschema)
   (paper "A4")
+  (wire (pts (xy 171.45 160.02) (xy 171.45 106.68))
+    (stroke (width 0) (type default))
+  )
+  (wire (pts (xy 167.64 34.29) (xy 167.64 58.42))
+    (stroke (width 0) (type default))
+  )
+  (wire (pts (xy 151.13 160.02) (xy 171.45 160.02))
+    (stroke (width 0) (type default))
+  )
+  (wire (pts (xy 180.34 34.29) (xy 167.64 34.29))
+    (stroke (width 0) (type default))
+  )
+  (wire (pts (xy 80.01 80.01) (xy 73.66 80.01))
+    (stroke (width 0) (type default))
+  )
+  (wire (pts (xy 87.63 106.68) (xy 80.01 106.68))
+    (stroke (width 0) (type default))
+  )
+  (wire (pts (xy 170.18 60.96) (xy 170.18 36.83))
+    (stroke (width 0) (type default))
+  )
+  (wire (pts (xy 167.64 58.42) (xy 151.13 58.42))
+    (stroke (width 0) (type default))
+  )
+  (wire (pts (xy 151.13 60.96) (xy 170.18 60.96))
+    (stroke (width 0) (type default))
+  )
+  (wire (pts (xy 80.01 106.68) (xy 80.01 80.01))
+    (stroke (width 0) (type default))
+  )
+  (wire (pts (xy 170.18 36.83) (xy 180.34 36.83))
+    (stroke (width 0) (type default))
+  )
+  (wire (pts (xy 171.45 106.68) (xy 200.66 106.68))
+    (stroke (width 0) (type default))
+  )
   (symbol (lib_id "knock:Module-knock-0.2") (at 187.96 114.3 0) (unit 1)
     (in_bom yes) (on_board yes) (dnp no) (fields_autoplaced)
@@
         (path "/10fbc709-889c-4565-8161-129ca9f0b73f"
           (reference "M4") (unit 1)
+        )
+      )
+    )
+  )
+  (symbol (lib_id "power:GND") (at 203.2 139.7 0) (unit 1)
+    (in_bom yes) (on_board yes) (dnp no) (fields_autoplaced)
+    (property "Reference" "#PWR03" (at 203.2 146.05 0)
+      (effects (font (size 1.27 1.27)) hide)
+    )
+    (property "Value" "GND" (at 203.2 144.78 0)
+      (effects (font (size 1.27 1.27)))
+    )
+    (property "Footprint" "" (at 203.2 139.7 0)
+      (effects (font (size 1.27 1.27)) hide)
+    )
+    (property "Datasheet" "" (at 203.2 139.7 0)
+      (effects (font (size 1.27 1.27)) hide)
+    )
+    (pin "1")
+    (instances
+      (project "EP91Starlet"
+        (path "/10fbc709-889c-4565-8161-129ca9f0b73f"
+          (reference "#PWR03") (unit 1)
+        )
+      )
+    )
+  )
+  (symbol (lib_id "power:GND") (at 228.6 49.53 0) (unit 1)
+    (in_bom yes) (on_board yes) (dnp no) (fields_autoplaced)
+    (property "Reference" "#PWR04" (at 228.6 55.88 0)
+      (effects (font (size 1.27 1.27)) hide)
+    )
+    (property "Value" "GND" (at 228.6 54.61 0)
+      (effects (font (size 1.27 1.27)))
+    )
+    (property "Footprint" "" (at 228.6 49.53 0)
+      (effects (font (size 1.27 1.27)) hide)
+    )
+    (property "Datasheet" "" (at 228.6 49.53 0)
+      (effects (font (size 1.27 1.27)) hide)
+    )
+    (pin "1")
+    (instances
+      (project "EP91Starlet"
+        (path "/10fbc709-889c-4565-8161-129ca9f0b73f"
+          (reference "#PWR04") (unit 1)
+        )
+      )
+    )
+  )
+  (symbol (lib_id "power:GND") (at 25.4 90.17 0) (unit 1)
+    (in_bom yes) (on_board yes) (dnp no) (fields_autoplaced)
+    (property "Reference" "#PWR01" (at 25.4 96.52 0)
+      (effects (font (size 1.27 1.27)) hide)
+    )
+    (property "Value" "GND" (at 25.4 95.25 0)
+      (effects (font (size 1.27 1.27)))
+    )
+    (property "Footprint" "" (at 25.4 90.17 0)
+      (effects (font (size 1.27 1.27)) hide)
+    )
+    (property "Datasheet" "" (at 25.4 90.17 0)
+      (effects (font (size 1.27 1.27)) hide)
+    )
+    (pin "1")
+    (instances
+      (project "EP91Starlet"
+        (path "/10fbc709-889c-4565-8161-129ca9f0b73f"
+          (reference "#PWR01") (unit 1)
+        )
+      )
+    )
+  )
+  (symbol (lib_id "power:GND") (at 87.63 175.26 0) (unit 1)
+    (in_bom yes) (on_board yes) (dnp no) (fields_autoplaced)
+    (property "Reference" "#PWR02" (at 87.63 181.61 0)
+      (effects (font (size 1.27 1.27)) hide)
+    )
+    (property "Value" "GND" (at 87.63 180.34 0)
+      (effects (font (size 1.27 1.27)))
+    )
+    (property "Footprint" "" (at 87.63 175.26 0)
+      (effects (font (size 1.27 1.27)) hide)
+    )
+    (property "Datasheet" "" (at 87.63 175.26 0)
+      (effects (font (size 1.27 1.27)) hide)
+    )
+    (pin "1")
+    (instances
+      (project "EP91Starlet"
+        (path "/10fbc709-889c-4565-8161-129ca9f0b73f"
+          (reference "#PWR02") (unit 1)
         )
       )
@@
     )
   )
-  (symbol (lib_id "vr-max9924:Module-vr-max9924-0.1") (at 187.96 81.28 0) (unit 1)
-    (in_bom yes) (on_board yes) (dnp no) (fields_autoplaced)
-    (property "Reference" "M3" (at 204.47 76.2 0)
-      (effects (font (size 1.27 1.27)))
-    )
-    (property "Value" "Module-vr-max9924-0.1" (at 204.47 78.74 0)
-      (effects (font (size 1.27 1.27)))
-    )
-    (property "Footprint" "0.3:vr-max9924" (at 213.36 80.01 0)
-      (effects (font (size 1.27 1.27)) hide)
-    )
-    (property "Datasheet" "" (at 187.96 81.28 0)
-      (effects (font (size 1.27 1.27)) hide)
-    )
+  (symbol (lib_id "vr-max9924:Module-vr-max9924-0.1") (at 33.02 77.47 0) (unit 1)
+    (in_bom yes) (on_board yes) (dnp no) (fields_autoplaced)
+    (property "Reference" "M3" (at 49.53 72.39 0)
+      (effects (font (size 1.27 1.27)))
+    )
+    (property "Value" "Module-vr-max9924-0.1" (at 49.53 74.93 0)
+      (effects (font (size 1.27 1.27)))
+    )
+    (property "Footprint" "0.3:vr-max9924" (at 58.42 76.2 0)
+      (effects (font (size 1.27 1.27)) hide)
+    )
+    (property "Datasheet" "" (at 33.02 77.47 0)
+      (effects (font (size 1.27 1.27)) hide)
+    )

Commit message: 65urft7ih
Parts:
- added M5: Module:mega-mcu100/0.3, hellen-one-mega-mcu100-0.3:mega-mcu100, symbol mega-mcu100:Module{colon}mega-mcu100/0.3
- added U1: ~, EP91Starlet:4EFE ECU Connector, symbol 4EFE ECU Connector:4EFE_ECU_Connector
Connections:
- net CAN+: now reaches M1.W12 (CAN1H)
- net CAN+: now also M2.W4 (CANH); no longer M2.W3 (CANL)
- net CAN-: now reaches M1.W13 (CAN1L)
- net CAN-: now also M2.W3 (CANL); no longer M2.W4 (CANH)
- removed net GND: M1.G (GND), M2.G (GND), M3.G (GND), M4.E2 (GND)
Changed lines of the file:
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@@
 (kicad_sch (version 20230121) (generator eeschema)
   (paper "A4")
+  (wire (pts (xy 165.1 60.96) (xy 165.1 34.29))
+    (stroke (width 0) (type default))
+  )
   (wire (pts (xy 171.45 160.02) (xy 171.45 106.68))
     (stroke (width 0) (type default))
   )
-  (wire (pts (xy 167.64 34.29) (xy 167.64 58.42))
+  (wire (pts (xy 167.64 36.83) (xy 180.34 36.83))
     (stroke (width 0) (type default))
   )
@@
     (stroke (width 0) (type default))
   )
-  (wire (pts (xy 180.34 34.29) (xy 167.64 34.29))
+  (wire (pts (xy 165.1 34.29) (xy 180.34 34.29))
     (stroke (width 0) (type default))
   )
@@
     (stroke (width 0) (type default))
   )
-  (wire (pts (xy 170.18 60.96) (xy 170.18 36.83))
-    (stroke (width 0) (type default))
-  )
-  (wire (pts (xy 167.64 58.42) (xy 151.13 58.42))
-    (stroke (width 0) (type default))
-  )
-  (wire (pts (xy 151.13 60.96) (xy 170.18 60.96))
+  (wire (pts (xy 167.64 58.42) (xy 167.64 36.83))
+    (stroke (width 0) (type default))
+  )
+  (wire (pts (xy 151.13 60.96) (xy 165.1 60.96))
     (stroke (width 0) (type default))
   )
@@
     (stroke (width 0) (type default))
   )
-  (wire (pts (xy 170.18 36.83) (xy 180.34 36.83))
+  (wire (pts (xy 151.13 58.42) (xy 167.64 58.42))
     (stroke (width 0) (type default))
   )
   (wire (pts (xy 171.45 106.68) (xy 200.66 106.68))
     (stroke (width 0) (type default))
+  )
+  (label "CAN-" (at 157.48 60.96 0) (fields_autoplaced)
+    (effects (font (size 1.27 1.27)) (justify left bottom))
+  )
+  (label "CAN+" (at 157.48 58.42 0) (fields_autoplaced)
+    (effects (font (size 1.27 1.27)) (justify left bottom))
+  )
+  (symbol (lib_id "4EFE ECU Connector:4EFE_ECU_Connector") (at 30.48 132.08 0) (unit 1)
+    (in_bom yes) (on_board yes) (dnp no) (fields_autoplaced)
+    (property "Reference" "U1" (at 46.99 111.76 0)
+      (effects (font (size 1.27 1.27)))
+    )
+    (property "Value" "~" (at 30.48 132.08 0)
+      (effects (font (size 1.27 1.27)))
+    )
+    (property "Footprint" "EP91Starlet:4EFE ECU Connector" (at 30.48 132.08 0)
+      (effects (font (size 1.27 1.27)) hide)
+    )
+    (property "Datasheet" "" (at 30.48 132.08 0)
+      (effects (font (size 1.27 1.27)) hide)
+    )
+    (pin "36")
+    (pin "30")
+    (pin "39")
+    (pin "27")
+    (pin "37")
+    (pin "40")
+    (pin "25")
+    (pin "26")
+    (pin "28")
+    (pin "7")
+    (pin "33")
+    (pin "42")
+    (pin "3")
+    (pin "41")
+    (pin "24")
+    (pin "35")
+    (pin "22")
+    (pin "4")
+    (pin "34")
+    (pin "8")
+    (pin "5")
+    (pin "6")
+    (pin "9")
+    (pin "31")
+    (pin "32")
+    (pin "23")
+    (pin "29")
+    (pin "38")
+    (pin "16")
+    (pin "17")
+    (pin "1")
+    (pin "11")
+    (pin "10")
+    (pin "12")
+    (pin "13")
+    (pin "15")
+    (pin "18")
+    (pin "19")
+    (pin "14")
+    (pin "2")
+    (pin "20")
+    (pin "21")
+    (instances
+      (project "EP91Starlet"
+        (path "/10fbc709-889c-4565-8161-129ca9f0b73f"
+          (reference "U1") (unit 1)
+        )
+      )
+    )
   )
   (symbol (lib_id "knock:Module-knock-0.2") (at 187.96 114.3 0) (unit 1)
@@
     )
   )
-  (symbol (lib_id "power:GND") (at 203.2 139.7 0) (unit 1)
+  (symbol (lib_id "mega-mcu100:Module{colon}mega-mcu100/0.3") (at 292.1 19.05 0) (unit 1)
     (in_bom yes) (on_board yes) (dnp no) (fields_autoplaced)
-    (property "Reference" "#PWR03" (at 203.2 146.05 0)
-      (effects (font (size 1.27 1.27)) hide)
-    )
-    (property "Value" "GND" (at 203.2 144.78 0)
-      (effects (font (size 1.27 1.27)))
-    )
-    (property "Footprint" "" (at 203.2 139.7 0)
-      (effects (font (size 1.27 1.27)) hide)
-    )
-    (property "Datasheet" "" (at 203.2 139.7 0)
-      (effects (font (size 1.27 1.27)) hide)
-    )
-    (pin "1")
+    (property "Reference" "M5" (at 326.39 11.43 0)
+      (effects (font (size 1.27 1.27)))
+    )
+    (property "Value" "Module:mega-mcu100/0.3" (at 326.39 13.97 0)
+      (effects (font (size 1.27 1.27)))
+    )
+    (property "Footprint" "hellen-one-mega-mcu100-0.3:mega-mcu100" (at 292.1 19.05 0)
+      (effects (font (size 1.27 1.27)) hide)
+    )
+    (property "Datasheet" "" (at 292.1 19.05 0)
+      (effects (font (size 1.27 1.27)) hide)
+    )
+    (property "PUBLISHER" "qwerty-off" (at 292.1 19.05 0)
+      (effects (font (size 1.27 1.27)) (justify left bottom) hide)
+    )
+    (property "SUPPLIER PART NUMBER 1" "*" (at 286.512 74.93 0)
+      (effects (font (size 1.27 1.27)) (justify left bottom) hide)
+    )
+    (property "SUPPLIER PART NUMBER 2" "*" (at 286.512 74.93 0)
+      (effects (font (size 1.27 1.27)) (justify left bottom) hide)
+    )
+    (property "SUPPLIER 1" "Mouser" (at 286.512 74.93 0)
+      (effects (font (size 1.27 1.27)) (justify left bottom) hide)
+    )
+    (property "SUPPLIER 2" "Digi-Key" (at 286.512 74.93 0)
+      (effects (font (size 1.27 1.27)) (justify left bottom) hide)
+    )
+    (property "FITTED" "False" (at 286.512 57.15 0)
+      (effects (font (size 1.27 1.27)) (justify left bottom) hide)
+    )
+    (property "PACKAGEREFERENCE" "" (at 286.512 57.15 0)
+      (effects (font (size 1.27 1.27)) (justify left bottom) hide)
+    )
+    (property "SUPPLIER 3" "LCSC" (at 286.512 57.15 0)
+      (effects (font (size 1.27 1.27)) (justify left bottom) hide)
+    )
+    (property "SUPPLIER PART NUMBER 3" "" (at 286.512 57.15 0)
+      (effects (font (size 1.27 1.27)) (justify left bottom) hide)
+    )
+    (property "TYPE" "Module" (at 286.512 57.15 0)
+      (effects (font (size 1.27 1.27)) (justify left bottom) hide)
+    )
+    (pin "E13")
+    (pin "E23")
+    (pin "N14")
+    (pin "E6")
+    (pin "E20")
+    (pin "E16")
+    (pin "N12")
+    (pin "N22")
+    (pin "N1")
+    (pin "N6")
+    (pin "S13")
+    (pin "E8")
+    (pin "N14a")
+    (pin "N15")
+    (pin "N17")
+    (pin "E5")
+    (pin "N19")
+    (pin "N23")
+    (pin "E12")
+    (pin "E10")
+    (pin "N8")
+    (pin "E21")
+    (pin "E11")
+    (pin "E2")
+    (pin "E7")
+    (pin "N21")
+    (pin "N5")
+    (pin "E19")
+    (pin "S11")
+    (pin "S16")
+    (pin "S14")
+    (pin "S18")
+    (pin "S19")
+    (pin "E1")
+    (pin "E3")
+    (pin "N2")
+    (pin "S12")
+    (pin "S17")
+    (pin "S20")
+    (pin "S10")
+    (pin "G")
+    (pin "S1")
+    (pin "E15")
+    (pin "E4")
+    (pin "N13")
+    (pin "N11")
+    (pin "N18")
+    (pin "E9")
+    (pin "N14b")
+    (pin "N7")
+    (pin "S15")
+    (pin "E22")
+    (pin "N4")
+    (pin "E17")
+    (pin "S2")
+    (pin "E18")
+    (pin "S21")
+    (pin "S22")
+    (pin "N10")
+    (pin "E14")
+    (pin "N16")
+    (pin "N20")
+    (pin "N3")
+    (pin "N9")
+    (pin "S7")
+    (pin "W6")
+    (pin "W14")
+    (pin "W7")
+    (pin "W9")
+    (pin "W2")
+    (pin "S3")
+    (pin "W1")
+    (pin "W5")
+    (pin "S5")
+    (pin "W11")
+    (pin "S6")
+    (pin "W12")
+    (pin "W13")
+    (pin "W8")
+    (pin "S4")
+    (pin "W10")
+    (pin "S8")
+    (pin "W4")
+    (pin "S9")
+    (pin "W3")
     (instances
       (project "EP91Starlet"
         (path "/10fbc709-889c-4565-8161-129ca9f0b73f"
-          (reference "#PWR03") (unit 1)
+          (reference "M5") (unit 1)
         )
       )
-    )
-  )
-  (symbol (lib_id "power:GND") (at 228.6 49.53 0) (unit 1)
-    (in_bom yes) (on_board yes) (dnp no) (fields_autoplaced)
-    (property "Reference" "#PWR04" (at 228.6 55.88 0)
-      (effects (font (size 1.27 1.27)) hide)
-    )
-    (property "Value" "GND" (at 228.6 54.61 0)
-      (effects (font (size 1.27 1.27)))
-    )
-    (property "Footprint" "" (at 228.6 49.53 0)
-      (effects (font (size 1.27 1.27)) hide)
-    )
-    (property "Datasheet" "" (at 228.6 49.53 0)
-      (effects (font (size 1.27 1.27)) hide)
-    )
-    (pin "1")
-    (instances
-      (project "EP91Starlet"
-        (path "/10fbc709-889c-4565-8161-129ca9f0b73f"
-          (reference "#PWR04") (unit 1)
-        )
-      )
-    )
-  )
-  (symbol (lib_id "power:GND") (at 25.4 90.17 0) (unit 1)
-    (in_bom yes) (on_board yes) (dnp no) (fields_autoplaced)
-    (property "Reference" "#PWR01" (at 25.4 96.52 0)
-      (effects (font (size 1.27 1.27)) hide)
-    )
-    (property "Value" "GND" (at 25.4 95.25 0)
-      (effects (font (size 1.27 1.27)))
-    )
-    (property "Footprint" "" (at 25.4 90.17 0)
-      (effects (font (size 1.27 1.27)) hide)
-    )
-    (property "Datasheet" "" (at 25.4 90.17 0)
-      (effects (font (size 1.27 1.27)) hide)
-    )
-    (pin "1")
-    (instances
-      (project "EP91Starlet"
-        (path "/10fbc709-889c-4565-8161-129ca9f0b73f"
-          (reference "#PWR01") (unit 1)
-        )
-      )
-    )
-  )
-  (symbol (lib_id "power:GND") (at 87.63 175.26 0) (unit 1)
-    (in_bom yes) (on_board yes) (dnp no) (fields_autoplaced)
-    (property "Reference" "#PWR02" (at 87.63 181.61 0)
-      (effects (font (size 1.27 1.27)) hide)
-    )
-    (property "Value" "GND" (at 87.63 180.34 0)
-      (effects (font (size 1.27 1.27)))
-    )
-    (property "Footprint" "" (at 87.63 175.26 0)
-      (effects (font (size 1.27 1.27)) hide)
-    )
-    (property "Datasheet" "" (at 87.63 175.26 0)
-      (effects (font (size 1.27 1.27)) hide)
-    )
-    (pin "1")
-    (instances
-      (project "EP91Starlet"
-        (path "/10fbc709-889c-4565-8161-129ca9f0b73f"
-          (reference "#PWR02") (unit 1)
-        )
-      )
