File: EP91Starlet.kicad_sch (KiCad schematic)
At the start: 16 parts, among them J1 Conn_02x04_Top_Bottom, J2 Conn_02x03_Top_Bottom, J3 Conn_02x10_Top_Bottom, J4 Conn_02x03_Odd_Even, J5 USB_B, J6 Conn_02x04_Top_Bottom, J7 Conn_02x03_Odd_Even, J8 Conn_01x02, M1 Module-vr-max9924-0.1, M2 Module-mega-mcu144-0.7, M3 Module-knock-0.2, M4 Module-wbo-0.5, M5 Module-vr-max9924-0.1, M6 Module-power_12and5V-0.3, M7 Module-can-0.1

Commit message: retry (last time i promise :))
Parts:
- removed J1, J6: Conn_02x04_Top_Bottom, Connector_Molex:Molex_Mini-Fit_Jr_5569-08A2_2x04_P4.20mm_Horizontal, symbol Connector_Generic:Conn_02x04_Top_Bottom
- removed J2: Conn_02x03_Top_Bottom, Connector_Molex:Molex_Mini-Fit_Jr_5569-06A2_2x03_P4.20mm_Horizontal, symbol Connector_Generic:Conn_02x03_Top_Bottom
- removed J3: Conn_02x10_Top_Bottom, Connector_Molex:Molex_Mini-Fit_Jr_5569-20A2_2x10_P4.20mm_Horizontal, symbol Connector_Generic:Conn_02x10_Top_Bottom
- removed J4, J7: Conn_02x03_Odd_Even, Connector_PinHeader_2.54mm:PinHeader_2x03_P2.54mm_Vertical, symbol Connector_Generic:Conn_02x03_Odd_Even
- removed J5: USB_B, footprints:USB_B, symbol Connector:USB_B
- removed J8: Conn_01x02, Connector_PinHeader_2.54mm:PinHeader_2x01_P2.54mm_Vertical, symbol Connector_Generic:Conn_01x02
- removed M1, M5: Module-vr-max9924-0.1, vrmax9924:vr-max9924, symbol vr-max9924:Module-vr-max9924-0.1
- removed M2: Module-mega-mcu144-0.7, megamcu144:mega-mcu144, symbol mega-mcu144:Module-mega-mcu144-0.7
- removed M3: Module-knock-0.2, knock:knock, symbol knock:Module-knock-0.2
- removed M4: Module-wbo-0.5, wbo:wbo, symbol wbo:Module-wbo-0.5
- removed M6: Module-power_12and5V-0.3, power5_12:power_12and5V, symbol power_12and5V:Module-power_12and5V-0.3
- removed M7: Module-can-0.1, can:can, symbol can:Module-can-0.1
- removed U7: ~, ul_175446-6:CONN_175446-6_TYCO_TYC, symbol 4EFE ECU Connector:4EFE_ECU_Connector
Connections:
- no-connect marks 30 -> 0
Other:
- removed sheet INJ4
- removed sheet LS_PROTECTED_2 A
- removed sheet LS_PROTECTED_2 B
- removed sheet LS_PROTECTED_2 C
- removed sheet LS_PROTECTED_2 D
- note removed: "5V out"

Commit message: update
Parts:
- added M1: Module-mega-mcu144-0.7, mega-mcu144:mega-mcu144, symbol mega-mcu144:Module-mega-mcu144-0.7
- added U1: ~, symbol VNLD5090-E:VNLD5090-E

Commit message: sync
Parts:
- removed U1: ~, symbol VNLD5090-E:VNLD5090-E
- added J1: 175446-6, 1754466, symbol 175446-6:175446-6
- added M2: Module-vr-max9924-0.1, hellen-one-vr-max9924-0.1:vr-max9924, symbol vr-max9924:Module-vr-max9924-0.1
- added M3: Module-vr-discrete-0.5, hellen-one-vr-discrete-0.5:vr-discrete, symbol vr-discrete:Module-vr-discrete-0.5
- added M4: Module-power_12and5V-0.3, hellen-one-power_12and5V-0.3:power_12and5V, symbol power_12and5V:Module-power_12and5V-0.3
- added M5: Module-wbo-0.5, hellen-one-wbo-0.5:wbo, symbol wbo:Module-wbo-0.5
- M1: footprint mega-mcu144:mega-mcu144 -> hellen-one-mega-mcu144-0.7:mega-mcu144
Connections:
- net MAP: now reaches M1.S21 (IN_MAP1)
- net MAP: now also J1.104 (PIM)
- net IN_CRANK: now reaches M1.S22 (IN_CRANK)
- net IN_CRANK: now also M2.E3 (OUT)
- net IN_CAM: now reaches M1.S24 (IN_CAM)
- net IN_CAM: now also M3.E3 (OUT)
- net AIR: now reaches M1.S26 (IN_IAT)
- net AIR: now also J1.105 (THA)
- net COOLANT: now reaches M1.S28 (IN_CLT)
- net COOLANT: now also J1.103 (THW)
- net TPS: now reaches M1.S30 (IN_TPS)
- net TPS: now also J1.117 (PSW)
- net SPARK1: now reaches M1.W11 (IGN1)
- net SPARK1: now also J1.106 (IGT)
- new net +12V_PERM: J1.2 (BATT), M4.V1 (V12_PERM)
- new net +12V_RAW: J1.9 (+B), M4.V2 (IN_VIGN), M4.V3 (V12_RAW)
- new net +5VP: J1.118 (VCC)
- new net CATCONVERTLIGHT: J1.11 (EGW)
- new net CHECKENGINELIGHT: J1.10 (W)
- new net GND: J1.113 (E01), J1.124 (E1), J1.MH1, J1.MH2, J1.MH3, M4.S1 (GND)
- new net GNDA: J1.116 (E2)
- new net IACCLOSE: J1.101 (RSC)
- new net IACOPEN: J1.114 (RSO)
- new net IDLESWITCH: J1.119 (IDL)
- new net INJ1: J1.112 (#10)
- new net INJ2: J1.125 (#20)
- new net VR-: J1.109 (NE-), M2.W1 (VR-/HALL), M3.W1 (VR-)
- new net VRCRANK+: J1.121 (NE), M2.W2 (VR+)
- no-connect marks 0 -> 10

Commit message: sync
Parts:
- added J2: Conn_02x15_Top_Bottom, Connector_PinHeader_2.54mm:PinHeader_2x15_P2.54mm_Vertical, symbol Connector_Generic:Conn_02x15_Top_Bottom
- added M6: Module-knock-0.2, hellen-one-knock-0.2:knock, symbol knock:Module-knock-0.2
- added R1, R2, R3, R4: 4.7k, symbol Device:R
- added U1, U2: VNLD5090-E, symbol VNLD5090-E:VNLD5090-E
- J1: footprint 1754466 -> 175446-6:1754466
- M1: footprint hellen-one-mega-mcu144-0.7:mega-mcu144 -> mega-mcu144:mega-mcu144
- M2: footprint hellen-one-vr-max9924-0.1:vr-max9924 -> vr-max9924:vr-max9924
- M3: footprint hellen-one-vr-discrete-0.5:vr-discrete -> vr-discrete:vr-discrete
- M4: footprint hellen-one-power_12and5V-0.3:power_12and5V -> power_12and5V:power_12and5V
- M5: footprint hellen-one-wbo-0.5:wbo -> wbo:wbo
Connections:
- net GND: now also R1.2, R2.2, R3.2, R4.2, U1.5 (SOURCE2), U1.7 (SOURCE1), U2.5 (SOURCE2), U2.7 (SOURCE1)
- net SPARK1: no longer M1.W11 (IGN1)
- net CHECKENGINE_IN: now reaches M1.E12 (OUT_IO2)
- net INJ2_IN: now reaches M1.E18 (OUT_INJ2)
- net INJ2_IN: now also R2.1, U1.3 (IN2)
- net INJ1_IN: now reaches M1.E19 (OUT_INJ1)
- net INJ1_IN: now also R1.1, U1.1 (IN1)
- net INJ3_IN: now reaches M1.E29 (OUT_INJ3)
- net INJ3_IN: now also R4.1, U2.1 (IN1)
- net INJ4_IN: now reaches M1.E30 (OUT_INJ4)
- net INJ4_IN: now also R3.1, U2.3 (IN2)
- net CHECKCAT_IN: now reaches M1.E6 (OUT_IO3)
- net FUELRELAY_IN: now reaches M1.E8 (OUT_IO1)
- net O2SENS: now reaches M1.S16 (IN_O2S)
- net O2SENS: now also J1.110 (OX)
- net SPARK2_OUT: now reaches M1.W10 (IGN2)
- net SPARK4_OUT: now reaches M1.W8 (IGN4)
- net SPARK3_OUT: now reaches M1.W9 (IGN3)
- net O2HEAT_OUT: now reaches J1.115 (HT)
- net FUELRELAY_OUT: now reaches J1.4 (FC)
- net CATCONVERTLIGHT renamed CHECKCAT_OUT
- net CHECKENGINELIGHT renamed CHECKENGINE_OUT
- new net INJ1_OUT: U1.8 (DRAIN1)
- new net INJ2_OUT: U1.6 (DRAIN2)
- new net INJ3_OUT: U2.8 (DRAIN1)
- new net INJ4_OUT: U2.6 (DRAIN2)
- new net SPARK1_OUT: M1.W11 (IGN1)
- no-connect marks 10 -> 14
Other:
- note added: "HOT LS (INJECTOR)"
- moved on the sheet: J1, M1

Commit message: sync
Parts:
- removed M5: Module-wbo-0.5, wbo:wbo, symbol wbo:Module-wbo-0.5
- added BT1: CR1220, kicad6-libraries:CR1220-2, symbol Device:Battery_Cell
- added D1, D2, D3, D4, D6, D7, D8, D9: B5819W, Diode_SMD:D_SOD-123, symbol Device:D
- added D5: 1N4148WS, Diode_SMD:D_SOD-323, symbol hellen-one-common:1N4148WS
- added M5: Module-wbo-0.6, wbo:wbo, symbol wbo:Module-wbo-0.6
- added Q2: BSS138, Package_TO_SOT_SMD:SOT-23, symbol Transistor_FET:BSS138
- added R10: 510R, Resistor_SMD:R_0402_1005Metric, symbol Device:R
- added R11, R12, R13, R14, R5, R6, R7, R8: 4.7k, Resistor_SMD:R_0402_1005Metric, symbol Device:R
- added R9: 10k, Resistor_SMD:R_0402_1005Metric, symbol Device:R
- added U3, U4, U5, U6: VNLD5090-E, VNLD5090-E:VNLD5090-E, symbol VNLD5090-E:VNLD5090-E
- M6: footprint hellen-one-knock-0.2:knock -> knock:knock
- R1, R2, R3, R4: footprint (none) -> Resistor_SMD:R_0402_1005Metric
- U1, U2: footprint (none) -> VNLD5090-E:VNLD5090-E
Connections:
- net +12V_RAW: now also D1.1 (K), D2.1 (K), D3.1 (K), D4.1 (K), D6.1 (K), D7.1 (K), D8.1 (K), D9.1 (K)
- net +5VP: now also M4.V4 (5VP)
- net CHECKENGINE_IN: now also R10.2
- net CHECKENGINE_OUT: now also Q2.3 (D)
- net FUELRELAY_IN: now also R5.1, U3.3 (IN2)
- net FUELRELAY_OUT: now also U3.8 (DRAIN1)
- net GND: now also M1.G (GND), M2.G (GND), M3.G (GND), M6.E2 (GND), BT1.2 (-), Q2.2 (S), R11.2, R12.2, R13.2, R14.2, R5.2, R6.2, R7.2, R8.2, R9.2, U3.5 (SOURCE2), U3.7 (SOURCE1), U4.5 (SOURCE2), U4.7 (SOURCE1), U5.5 (SOURCE2), U5.7 (SOURCE1), U6.5 (SOURCE2), U6.7 (SOURCE1)
- net GNDA: now also M1.E39 (GNDA), M1.W1 (GNDA)
- net LS3_IN: now reaches M1.E14 (OUT_PWM5)
- net LS3_IN: now also R14.1, U6.1 (IN1)
- net LS2_IN: now reaches M1.E15 (OUT_PWM4)
- net LS2_IN: now also R11.1, U5.3 (IN2)
- net LS1_IN: now reaches M1.E16 (OUT_PWM3)
- net LS1_IN: now also R12.1, U5.1 (IN1)
- net IACOPEN_IN: now reaches M1.E17 (OUT_PWM2)
- net IACOPEN_IN: now also R7.1, U4.3 (IN2)
- net FANRELAY_IN: now reaches M1.E21 (OUT_IO4)
- net FANRELAY_IN: now also R6.1, U3.1 (IN1)
- net LS4_IN: now reaches M1.E26 (OUT_PWM6)
- net LS4_IN: now also R13.1, U6.3 (IN2)
- net IACCLOSE_IN: now reaches M1.E27 (OUT_PWM1)
- net IACCLOSE_IN: now also R8.1, U4.1 (IN1)
- net THRESH: now reaches M1.E28 (OUT_PWM8)
- net THRESH: now also M3.E1 (Thresh_IN)
- net +5VA: now reaches M1.E38 (V5A_SWITCHABLE)
- net +5VA: now also M1.N30 (V5A_SWITCHABLE), M1.W2 (V5A_SWITCHABLE), M2.E4 (V5_IN), M3.E4 (V5_IN), M6.E1 (V5A)
- net +3.3V: now reaches M1.N22 (V33)
- net +3.3V: now also M1.N32 (V33)
- net VIGN: now reaches M1.N26 (IN_VIGN)
- net VIGN: now also M4.E3 (VIGN)
- net VBAT: now reaches M1.N27 (VBAT)
- net VBAT: now also M4.E1 (VBAT), D5.1 (K)
- net +3.3VA: now reaches M1.N28 (V33_SWITCHABLE)
- net PWR_EN: now reaches M1.N29 (OUT_PWR_EN)
- net PWR_EN: now also M4.E5 (EN_5VP)
- net +5V: now reaches M1.N31 (VCC)
- net +5V: now also M4.E4 (V5)
- net D4_IN: now reaches M1.S1 (IN_D4)
- net D4_IN: now also J2.8 (Pin_8)
- net AUX4: now reaches M1.S10 (IN_AUX4)
- net AUX3: now reaches M1.S11 (IN_AUX3)
- net AUX2: now reaches M1.S12 (IN_AUX2)
- net AUX1: now reaches M1.S13 (IN_AUX1)
- net D3_IN: now reaches M1.S2 (IN_D3)
- net D3_IN: now also J2.7 (Pin_7)
- net KNOCK_PROCESSED: now reaches M1.S23 (IN_KNOCK)
- net KNOCK_PROCESSED: now also M6.E3 (OUT_KNOCK)
- net VSS: now reaches M1.S25 (IN_VSS)
- net VSS: now also J1.13 (SPD)
- net D2_IN: now reaches M1.S3 (IN_D2)
- net D2_IN: now also J2.6 (Pin_6)
- net VREF1: now reaches M1.S35 (VREF1)
- net VREF1: now also M6.W2 (VREF)
- net D1_IN: now reaches M1.S4 (IN_D1)
- net D1_IN: now also J2.5 (Pin_5)
- net LS4_OUT: now reaches J2.1 (Pin_1)
- net LS4_OUT: now also D8.2 (A), D9.2 (A), U6.6 (DRAIN2)
- net LS3_OUT: now reaches J2.2 (Pin_2)
- net LS3_OUT: now also U6.8 (DRAIN1)
- net LS2_OUT: now reaches J2.3 (Pin_3)
- net LS2_OUT: now also D6.2 (A), D7.2 (A), U5.6 (DRAIN2)
- net LS1_OUT: now reaches J2.4 (Pin_4)
- net LS1_OUT: now also U5.8 (DRAIN1)
- net KNOCK_RAW: now reaches J2.9 (Pin_9)
- net KNOCK_RAW: now also M6.W1 (IN_KNOCK)
- net FANRELAY_OUT: now reaches J1.120 (FAN)
- net FANRELAY_OUT: now also D1.2 (A), D2.2 (A), U3.6 (DRAIN2)
- net CHECKCAT_OUT: no longer names the net of J1.11 (EGW)
- net IACCLOSE renamed IACCLOSE_OUT
- net IACCLOSE_OUT: now also U4.8 (DRAIN1)
- net IACOPEN renamed IACOPEN_OUT
- net IACOPEN_OUT: now also D3.2 (A), D4.2 (A), U4.6 (DRAIN2)
- net IN_CAM renamed CAM
- net IN_CRANK renamed CRANK
- new net: Q2.1 (G), R10.1, R9.1
- new net: BT1.1 (+), D5.2 (A)
- no-connect marks 14 -> 24
Other:
- note added: "Extra LS"
- note added: "Hot LS (Injectors)"
- note added: "Protected LS (Relays/Solenoids)"
- note added: "Weak LS (Check Engine Light)"
- note removed: "HOT LS (INJECTOR)"
- moved on the sheet: J1, J2, M1, M2, M3, M4, M6
