File: EP91Starlet.kicad_sch (KiCad schematic)
At the start: 42 parts, among them J1 175446-6, J2 Extra Inputs (2.54mm Pin Head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, J3 TE_6473423-1_26p, M1 Module-mega-mcu144-0.7, M2 Module-vr-max9924-0.1, M3 Module-vr-discrete-0.5, M4 Module-power_12and5V-0.3, M5 Module-wbo-0.6, M6 Module-knock-0.2, M7 Module-can-0.1, Q2 BSS138, U1 VNLD5090-E, U2 VNLD5090-E, U3 VNLD5090-E, U4 VNLD5090-E, U5 VNLD5090-E, U6 VNLD5090-E

Commit message: sync
Parts:
- removed J2: Extra Inputs (2.54mm Pin Header), Connector_PinHeader_2.54mm:PinHeader_2x15_P2.54mm_Vertical, symbol Connector_Generic:Conn_02x15_Top_Bottom
- removed J3: TE_6473423-1_26p, TE:6473423-1, symbol Connectors:TE_6473423-1_26p
- added J2: USB_B, kicad6-libraries:USB_B, symbol misc:USB_B
- added J3, J4, J5, J6: Conn_02x10_Odd_Even, symbol Connector_Generic:Conn_02x10_Odd_Even
- added U7: ULN2003A, symbol Transistor_Array:ULN2003A
- J1: footprint 175446-6:1754466 -> TE-175446-6:1754466
- M1: footprint mega-mcu144:mega-mcu144 -> hellen-one-mega-mcu144:mega-mcu144
- M2: footprint vr-max9924:vr-max9924 -> hellen-one-vr-max9924:vr-max9924
- M3: footprint vr-discrete:vr-discrete -> hellen-one-vr-discrete:vr-discrete
- M4: footprint power_12and5V:power_12and5V -> hellen-one-power_12and5V:power_12and5V
- M5: footprint wbo:wbo -> hellen-one-wbo:wbo
- M6: footprint knock:knock -> hellen-one-knock:knock
- M7: footprint can:can -> hellen-one-can:can
- TP1: footprint (none) -> hellen-one-vr-max9924:vr-max9924
Connections:
- net CHECKCAT_IN is gone; now on net FANRELAY_IN: M1.E6 (OUT_IO3)
- net +12V_RAW: now also J6.10 (Pin_10), U7.9 (COM)
- net +5VP: now also J3.18 (Pin_18), J4.1 (Pin_1), J5.1 (Pin_1)
- net AT1: now also J4.14 (Pin_14)
- net AT2: now also J4.16 (Pin_16)
- net AUX1: now also J4.3 (Pin_3)
- net AUX2: now also J4.5 (Pin_5)
- net AUX3: now also J4.7 (Pin_7)
- net AUX4: now also J4.9 (Pin_9)
- net CAN1+: no longer M1.W12 (CANH)
- net CAN1-: no longer M1.W13 (CANL)
- net D1_IN: now also J5.3 (Pin_3)
- net D2_IN: now also J5.5 (Pin_5)
- net D3_IN: now also J5.7 (Pin_7)
- net D4_IN: now also J5.9 (Pin_9)
- net FANRELAY_IN: no longer M1.E21 (OUT_IO4)
- net GND: now also J2.4 (GND), J2.5 (Shield), J3.20 (Pin_20), J5.2 (Pin_2), J6.12 (Pin_12), U7.8 (GND)
- net GNDA: now also J4.2 (Pin_2)
- net KNOCK_RAW: now also J4.11 (Pin_11)
- net LS1_OUT: now also J6.2 (Pin_2)
- net LS2_OUT: now also J6.4 (Pin_4)
- net LS3_OUT: now also J6.6 (Pin_6)
- net LS4_OUT: now also J6.8 (Pin_8)
- net MAP2: now also J4.4 (Pin_4)
- net MAP3: now also J4.6 (Pin_6)
- net O2S2: now also J4.18 (Pin_18)
- net PPS: now also J4.8 (Pin_8)
- net PPS2: now also J4.10 (Pin_10)
- net RES1: now also J5.11 (Pin_11)
- net RES2: now also J5.13 (Pin_13)
- net RES3: now also J5.15 (Pin_15)
- net SENS1: now also J5.4 (Pin_4)
- net SENS2: now also J5.6 (Pin_6)
- net SENS3: now also J5.8 (Pin_8)
- net SENS4: now also J5.10 (Pin_10)
- net TPS2: now also J4.12 (Pin_12)
- net at M1.N2 (USBM): now also J2.2 (D-)
- net at M1.N3 (USBP): now also J2.3 (D+)
- net at M1.N4 (VBUS): now also J2.1 (VBUS)
- net 5V_OUT8: now reaches M1.W4 (IGN8)
- net 5V_OUT8: now also J3.15 (Pin_15)
- net 5V_OUT7: now reaches M1.W5 (IGN7)
- net 5V_OUT7: now also J3.13 (Pin_13)
- net 5V_OUT6: now reaches M1.W6 (IGN6)
- net 5V_OUT6: now also J3.11 (Pin_11)
- net 5V_OUT5: now reaches M1.W7 (IGN5)
- net 5V_OUT5: now also J3.9 (Pin_9)
- net CAN2+ renamed CAN1_HIGH
- net CAN1_HIGH: now also J3.2 (Pin_2)
- net CAN2- renamed CAN1_LOW
- net CAN1_LOW: now also J3.4 (Pin_4)
- net INJ1_IN renamed LS1_HOT_IN
- net INJ1_OUT renamed LS1_HOT_OUT
- net LS1_HOT_OUT: now also J6.1 (Pin_1)
- net INJ2_IN renamed LS2_HOT_IN
- net INJ2_OUT renamed LS2_HOT_OUT
- net LS2_HOT_OUT: now also J6.3 (Pin_3)
- net INJ3_IN renamed LS4_HOT_IN
- net LS4_HOT_IN: now also M1.E30 (OUT_INJ4); no longer M1.E29 (OUT_INJ3)
- net INJ3_OUT renamed LS4_HOT_OUT
- net LS4_HOT_OUT: now also J6.7 (Pin_7)
- net INJ4_IN renamed LS3_HOT_IN
- net LS3_HOT_IN: now also M1.E29 (OUT_INJ3); no longer M1.E30 (OUT_INJ4)
- net INJ4_OUT renamed LS3_HOT_OUT
- net LS3_HOT_OUT: now also J6.5 (Pin_5)
- net IO1: no longer names the net of M1.N16 (IO1)
- net IO2: no longer names the net of M1.N19 (IO2)
- net IO3: no longer names the net of M1.N21 (IO3)
- net IO4: no longer names the net of M1.N20 (IO4)
- net IO5: no longer names the net of M1.N23 (IO5)
- net IO6: no longer names the net of M1.E35 (IO6)
- net SPARK1_OUT renamed 5V_OUT1
- net 5V_OUT1: now also J3.1 (Pin_1)
- net SPARK2_OUT renamed 5V_OUT2
- net 5V_OUT2: now also J3.3 (Pin_3)
- net SPARK3_OUT renamed 5V_OUT3
- net 5V_OUT3: now also J3.5 (Pin_5)
- net SPARK4_OUT renamed 5V_OUT4
- net 5V_OUT4: now also J3.7 (Pin_7)
- new net CAN2_HIGH: J3.6 (Pin_6), M1.W12 (CANH)
- new net CAN2_LOW: J3.8 (Pin_8), M1.W13 (CANL)
- new net DC1+: J6.9 (Pin_9)
- new net DC1-: J6.11 (Pin_11)
- no-connect marks 26 -> 28
Other:
- note added: "2.54mm Pin Header"
- note added: "Extra Analogue / Switch Inputs (2.54mm Pin Header) AUX1-4 has EXTI (Can do event input)"
- note added: "Extra Event / Switch Inputs (2.54mm Pin Header) DC1-4 Is fastest, ideal for PWM input (flex fuel, etc)"
- note added: "Extra LS Drivers"
- note added: "Extra Outputs (AMP Superseal 1.0 26 Pin) LS_OUT are 3.5A lowside drivers intended e.g. relay, 3.5A continuous, has external flyback diode LS_HOT_OUT are lowside drivers e.g. injector 3.5A continuous, has no flyback diode DC is H-bridge e.g. ETB, EWG, any DC motor 6A continuous 5V_OUT are 5V LOGIC Outputs e.g. Smart coils 24mA source/sink LS_HOT1-2 ALSO CONNECTED TO BATCH FIRE PINS ON STOCK HARNES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"
- note added: "Molex Mini-Fit Jr. Socket"
- note added: "Stock Harness ECU Connector (PNP)"
- note removed: "Extra LS"
- moved on the sheet: D6, D7, D8, D9, J1, M3, M4, M5, M6, R11, R12, R13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

Commit message: sync
Parts:
- removed J3, J4, J5, J6: Conn_02x10_Odd_Even, symbol Connector_Generic:Conn_02x10_Odd_Even
- removed TP1: TestPoint, hellen-one-vr-max9924:vr-max9924, symbol Connector:TestPoint
- removed U7: ULN2003A, symbol Transistor_Array:ULN2003A
- added F1: Fuse, Fuse:Fuse_1206_3216Metric_Pad1.42x1.75mm_HandSolder, symbol Device:Fuse
- added J3, J5: Conn_01x02, Connector_PinHeader_2.54mm:PinHeader_1x02_P2.54mm_Vertical, symbol Connector_Generic:Conn_01x02
- added J6: Conn_02x03_Top_Bottom, Connector_Molex:Molex_Mini-Fit_Jr_5566-06A_2x03_P4.20mm_Vertical, symbol Connector_Generic:Conn_02x03_Top_Bottom
- added J7: Conn_02x20_Odd_Even, Connector_IDC:IDC-Header_2x20_P2.54mm_Vertical, symbol Connector_Generic:Conn_02x20_Odd_Even
- added J9: Conn_02x06_Top_Bottom, Connector_Molex:Molex_Mini-Fit_Jr_5566-12A_2x06_P4.20mm_Vertical, symbol Connector_Generic:Conn_02x06_Top_Bottom
Connections:
- net CAN1+ is gone; now on net CAN1_HIGH: M5.W4 (CANH)
- net CAN1- is gone; now on net CAN1_LOW: M5.W3 (CANL)
- net INJ1 is gone; now on net LS1_HOT_OUT: J1.112 (#10)
- net INJ2 is gone; now on net LS2_HOT_OUT: J1.125 (#20)
- net SPARK1 is gone; now on net 5V_OUT1: J1.106 (IGT)
- net +12V_RAW: now also F1.1, J9.5 (Pin_5)
- net +5VP: now also J7.1 (Pin_1), J7.27 (Pin_27), J7.29 (Pin_29), J7.3 (Pin_3)
- net 5V_OUT1: now also J7.31 (Pin_31)
- net 5V_OUT2: now also J7.33 (Pin_33)
- net 5V_OUT3: now also J7.35 (Pin_35)
- net 5V_OUT4: now also J7.37 (Pin_37)
- net AT1: now also J7.13 (Pin_13)
- net AT2: now also J7.15 (Pin_15)
- net AUX1: now also J7.5 (Pin_5)
- net AUX2: now also J7.7 (Pin_7)
- net AUX3: now also J7.9 (Pin_9)
- net AUX4: now also J7.11 (Pin_11)
- net CAN1_HIGH: now also J7.32 (Pin_32)
- net CAN1_LOW: now also J7.34 (Pin_34)
- net CAN2_HIGH: now also J7.36 (Pin_36)
- net CAN2_LOW: now also J7.38 (Pin_38)
- net D1_IN: now also J7.25 (Pin_25)
- net D2_IN: now also J7.23 (Pin_23)
- net D3_IN: now also J7.21 (Pin_21)
- net D4_IN: now also J7.19 (Pin_19)
- net DC1+: now also J9.11 (Pin_11)
- net DC1-: now also J9.12 (Pin_12)
- net FANRELAY_IN: now also M1.E21 (OUT_IO4); no longer M1.E6 (OUT_IO3)
- net GND: now also J5.2 (Pin_2), J7.28 (Pin_28), J7.30 (Pin_30), J9.6 (Pin_6)
- net GNDA: now also J7.2 (Pin_2), J7.4 (Pin_4)
- net LS1_HOT_OUT: now also J9.4 (Pin_4)
- net LS1_OUT: now also J9.7 (Pin_7)
- net LS2_HOT_OUT: now also J9.3 (Pin_3)
- net LS2_OUT: now also J9.8 (Pin_8)
- net LS3_HOT_IN: now also R4.1, U2.1 (IN1); no longer R3.1, U2.3 (IN2)
- net LS3_HOT_OUT: now also U2.8 (DRAIN1), J9.2 (Pin_2); no longer U2.6 (DRAIN2)
- net LS3_OUT: now also J9.9 (Pin_9)
- net LS4_HOT_IN: now also R3.1, U2.3 (IN2); no longer R4.1, U2.1 (IN1)
- net LS4_HOT_OUT: now also U2.6 (DRAIN2), J9.1 (Pin_1); no longer U2.8 (DRAIN1)
- net LS4_OUT: now also J9.10 (Pin_10)
- net MAP2: now also J7.6 (Pin_6)
- net MAP3: now also J7.8 (Pin_8)
- net O2S2: now also J7.16 (Pin_16)
- net PPS: now also J7.10 (Pin_10)
- net PPS2: now also J7.12 (Pin_12)
- net RES1: now also J7.17 (Pin_17)
- net RES2: now also J7.18 (Pin_18); no longer M1.S14 (IN_RES2)
- net SENS1: now also J7.26 (Pin_26)
- net SENS2: now also J7.24 (Pin_24)
- net SENS3: now also J7.22 (Pin_22)
- net SENS4: now also J7.20 (Pin_20)
- net TPS2: now also J7.14 (Pin_14)
- net VREF1: now also M1.S5 (VREF2); no longer M1.S35 (VREF1)
- net PG: now reaches M4.E6 (PG_5VP)
- net PG: now also M1.N13 (SPI3_MOSI)
- net DC Driver 1/PWM: now reaches M1.E14 (OUT_PWM5)
- net DC Driver 1/DIS: now reaches M1.E7 (OUT_IO5)
- net EGT/SPI_CS: now reaches M1.N10 (SPI3_CS)
- net EGT/SPI_SCK: now reaches M1.N11 (SPI3_SCK)
- net EGT/SPI_SO: now reaches M1.N12 (SPI3_MISO)
- net KNOCK_RAW: no longer names the net of M6.W1 (IN_KNOCK)
- net KNOCK_RAW: now also J5.1 (Pin_1)
- new net DC Driver 1/DIR: M1.E6 (OUT_IO3)
- new net DC Driver 1/PWR: F1.2
- new net EGT/T+: J3.1 (Pin_1)
- new net EGT/T-: J3.2 (Pin_2)
Other:
- added sheet DC Driver 1 (DC_MOTOR_0.1.kicad_sch)
- added sheet EGT (EGT.kicad_sch)
- note removed: "2.54mm Pin Header"
- moved on the sheet: M5

Commit message: sync
Parts:
- M1: footprint hellen-one-mega-mcu144:mega-mcu144 -> hellen-one-mega-mcu144-0.7:mega-mcu144
- M2: footprint hellen-one-vr-max9924:vr-max9924 -> hellen-one-vr-max9924-0.3:vr-max9924
- M3: footprint hellen-one-vr-discrete:vr-discrete -> hellen-one-vr-discrete-0.5:vr-discrete
- M5: footprint hellen-one-wbo:wbo -> hellen-one-wbo-0.6:wbo
- M6: footprint hellen-one-knock:knock -> hellen-one-knock-0.2:knock
- M7: footprint hellen-one-can:can -> hellen-one-can-0.1:can
Connections:
- net +12V_RAW: now also J9.1 (Pin_1); no longer J9.5 (Pin_5)
- net GND: now also J9.2 (Pin_2); no longer J9.6 (Pin_6)
- net LS1_HOT_OUT: now also J9.6 (Pin_6); no longer J9.4 (Pin_4)
- net LS2_HOT_OUT: now also J9.5 (Pin_5); no longer J9.3 (Pin_3)
- net LS3_HOT_OUT: now also J9.4 (Pin_4); no longer J9.2 (Pin_2)
- net LS4_HOT_OUT: now also J9.3 (Pin_3); no longer J9.1 (Pin_1)
Changed lines of the file:
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@@
 	(wire
 		(pts
+			(xy 307.34 110.49) (xy 320.04 110.49)
+		)
+		(stroke
+			(width 0)
+			(type default)
+		)
+	)
+	(wire
+		(pts
 			(xy 252.73 101.6) (xy 255.27 101.6)
 		)
@@
 		)
 	)
-	(label "LS2_HOT_OUT"
-		(at 320.04 113.03 180)
-		(effects
-			(font
-				(size 1.27 1.27)
-			)
-			(justify right bottom)
-		)
-	)
 	(label "MAP2"
 		(at 382.27 97.79 0)
@@
 		)
 	)
+	(label "LS1_HOT_OUT"
+		(at 320.04 120.65 180)
+		(effects
+			(font
+				(size 1.27 1.27)
+			)
+			(justify right bottom)
+		)
+	)
 	(label "LS4_HOT_IN"
 		(at 67.31 58.42 0)
@@
 		)
 	)
-	(label "LS3_HOT_OUT"
-		(at 320.04 110.49 180)
-		(effects
-			(font
-				(size 1.27 1.27)
-			)
-			(justify right bottom)
-		)
-	)
 	(label "CAN1_LOW"
 		(at 382.27 133.35 0)
@@
 		)
 	)
-	(label "LS4_HOT_OUT"
-		(at 320.04 107.95 180)
-		(effects
-			(font
-				(size 1.27 1.27)
-			)
-			(justify right bottom)
-		)
-	)
 	(label "TPS2"
 		(at 190.5 147.32 180)
@@
 		)
 	)
+	(label "LS4_HOT_OUT"
+		(at 320.04 113.03 180)
+		(effects
+			(font
+				(size 1.27 1.27)
+			)
+			(justify right bottom)
+		)
+	)
 	(label "D2_IN"
 		(at 369.57 120.65 180)
@@
 		)
 	)
-	(label "LS1_HOT_OUT"
-		(at 320.04 115.57 180)
-		(effects
-			(font
-				(size 1.27 1.27)
-			)
-			(justify right bottom)
-		)
-	)
 	(label "IACOPEN_IN"
 		(at 82.55 139.7 0)
@@
 		)
 	)
+	(label "LS3_HOT_OUT"
+		(at 320.04 115.57 180)
+		(effects
+			(font
+				(size 1.27 1.27)
+			)
+			(justify right bottom)
+		)
+	)
 	(label "PPS"
 		(at 382.27 102.87 0)
@@
 		)
 	)
+	(label "LS2_HOT_OUT"
+		(at 320.04 118.11 180)
+		(effects
+			(font
+				(size 1.27 1.27)
+			)
+			(justify right bottom)
+		)
+	)
 	(label "LS2_HOT_IN"
 		(at 67.31 29.21 0)
@@
 			)
 		)
-		(property "Footprint" "hellen-one-can:can"
+		(property "Footprint" "hellen-one-can-0.1:can"
 			(at 276.86 15.24 0)
 			(effects
@@
 	)
 	(symbol
+		(lib_id "hellen-one-common:+12V_RAW")
+		(at 320.04 107.95 90)
+		(mirror x)
+		(unit 1)
+		(exclude_from_sim no)
+		(in_bom yes)
+		(on_board yes)
+		(dnp no)
+		(fields_autoplaced yes)
+		(property "Reference" "#PWR65"
+			(at 323.85 107.95 0)
+			(effects
+				(font
+					(size 1.27 1.27)
+				)
+				(hide yes)
+			)
+		)
+		(property "Value" "+12V_RAW"
+			(at 316.23 107.9499 90)
+			(effects
+				(font
+					(size 1.27 1.27)
+				)
+				(justify left)
+			)
+		)
+		(property "Footprint" ""
+			(at 320.04 107.95 0)
+			(effects
+				(font
+					(size 1.27 1.27)
+				)
+				(hide yes)
+			)
+		)
+		(property "Datasheet" ""
+			(at 320.04 107.95 0)
+			(effects
+				(font
+					(size 1.27 1.27)
+				)
+				(hide yes)
+			)
+		)
+		(property "Description" "Power symbol creates a global label with name \"+12V_RAW\""
+			(at 320.04 107.95 0)
+			(effects
+				(font
+					(size 1.27 1.27)
+				)
+				(hide yes)
+			)
+		)
+		(pin "1"
+		)
+		(instances
+			(project "EP91Starlet"
+				(path "/10fbc709-889c-4565-8161-129ca9f0b73f"
+					(reference "#PWR65")
+					(unit 1)
+				)
+			)
+		)
+	)
+	(symbol
 		(lib_id "Device:R")
 		(at 69.85 199.39 0)
@@
 			)
 		)
-		(property "Footprint" "hellen-one-mega-mcu144:mega-mcu144"
+		(property "Footprint" "hellen-one-mega-mcu144-0.7:mega-mcu144"
 			(at 190.5 20.32 0)
 			(effects
@@
 			)
 		)
-		(property "Footprint" "hellen-one-wbo:wbo"
+		(property "Footprint" "hellen-one-wbo-0.6:wbo"
 			(at 267.97 317.5 0)
 			(effects
@@
 	)
 	(symbol
+		(lib_id "power:GND")
+		(at 307.34 110.49 270)
+		(mirror x)
+		(unit 1)
+		(exclude_from_sim no)
+		(in_bom yes)
+		(on_board yes)
+		(dnp no)
+		(property "Reference" "#PWR67"
+			(at 300.99 110.49 0)
+			(effects
+				(font
+					(size 1.27 1.27)
+				)
+				(hide yes)
+			)
+		)
+		(property "Value" "GND"
+			(at 302.26 110.49 90)
+			(effects
+				(font
+					(size 1.27 1.27)
+				)
+			)
+		)
+		(property "Footprint" ""
+			(at 307.34 110.49 0)
+			(effects
+				(font
+					(size 1.27 1.27)
+				)
+				(hide yes)
+			)
+		)
+		(property "Datasheet" ""
+			(at 307.34 110.49 0)
+			(effects
+				(font
+					(size 1.27 1.27)
+				)
+				(hide yes)
+			)
+		)
+		(property "Description" "Power symbol creates a global label with name \"GND\" , ground"
+			(at 307.34 110.49 0)
+			(effects
+				(font
+					(size 1.27 1.27)
+				)
+				(hide yes)
+			)
+		)
+		(pin "1"
+		)
+		(instances
+			(project "EP91Starlet"
+				(path "/10fbc709-889c-4565-8161-129ca9f0b73f"
+					(reference "#PWR67")
+					(unit 1)
+				)
+			)
+		)
+	)
+	(symbol
 		(lib_id "Device:R")
 		(at 81.28 111.76 0)
@@
 			)
 		)
-		(property "Footprint" "hellen-one-vr-max9924:vr-max9924"
+		(property "Footprint" "hellen-one-vr-max9924-0.3:vr-max9924"
 			(at 63.5 254 0)
 			(effects
@@
 	)
 	(symbol
-		(lib_id "power:GND")
-		(at 320.04 120.65 270)
-		(mirror x)
-		(unit 1)
-		(exclude_from_sim no)
-		(in_bom yes)
-		(on_board yes)
-		(dnp no)
-		(property "Reference" "#PWR67"
-			(at 313.69 120.65 0)
-			(effects
-				(font
-					(size 1.27 1.27)
-				)
-				(hide yes)
-			)
-		)
-		(property "Value" "GND"
-			(at 314.96 120.65 90)
-			(effects
-				(font
-					(size 1.27 1.27)
-				)
-			)
-		)
-		(property "Footprint" ""
-			(at 320.04 120.65 0)
-			(effects
-				(font
-					(size 1.27 1.27)
-				)
-				(hide yes)
-			)
-		)
-		(property "Datasheet" ""
-			(at 320.04 120.65 0)
-			(effects
-				(font
-					(size 1.27 1.27)
-				)
-				(hide yes)
-			)
-		)
-		(property "Description" "Power symbol creates a global label with name \"GND\" , ground"
-			(at 320.04 120.65 0)
-			(effects
-				(font
-					(size 1.27 1.27)
-				)
-				(hide yes)
-			)
-		)
-		(pin "1"
-		)
-		(instances
-			(project "EP91Starlet"
-				(path "/10fbc709-889c-4565-8161-129ca9f0b73f"
-					(reference "#PWR67")
-					(unit 1)
-				)
-			)
-		)
-	)
-	(symbol
 		(lib_id "power:+5VA")
 		(at 138.43 316.23 0)
@@
 	(symbol
 		(lib_id "hellen-one-common:+12V_RAW")
-		(at 320.04 118.11 90)
-		(mirror x)
-		(unit 1)
-		(exclude_from_sim no)
-		(in_bom yes)
-		(on_board yes)
-		(dnp no)
-		(fields_autoplaced yes)
-		(property "Reference" "#PWR65"
-			(at 323.85 118.11 0)
-			(effects
-				(font
-					(size 1.27 1.27)
-				)
-				(hide yes)
-			)
-		)
-		(property "Value" "+12V_RAW"
-			(at 316.23 118.1099 90)
-			(effects
-				(font
-					(size 1.27 1.27)
-				)
-				(justify left)
-			)
-		)
-		(property "Footprint" ""
-			(at 320.04 118.11 0)
-			(effects
-				(font
-					(size 1.27 1.27)
-				)
-				(hide yes)
-			)
-		)
-		(property "Datasheet" ""
-			(at 320.04 118.11 0)
-			(effects
-				(font
-					(size 1.27 1.27)
-				)
-				(hide yes)
-			)
-		)
-		(property "Description" "Power symbol creates a global label with name \"+12V_RAW\""
-			(at 320.04 118.11 0)
-			(effects
-				(font
-					(size 1.27 1.27)
-				)
-				(hide yes)
-			)
-		)
-		(pin "1"
-		)
-		(instances
-			(project "EP91Starlet"
-				(path "/10fbc709-889c-4565-8161-129ca9f0b73f"
-					(reference "#PWR65")
-					(unit 1)
-				)
-			)
-		)
-	)
-	(symbol
-		(lib_id "hellen-one-common:+12V_RAW")
 		(at 38.1 215.9 0)
 		(unit 1)
@@
 			)
 		)
-		(property "Footprint" "hellen-one-vr-discrete:vr-discrete"
+		(property "Footprint" "hellen-one-vr-discrete-0.5:vr-discrete"
 			(at 63.5 275.59 0)
 			(effects
@@
 			)
 		)
-		(property "Footprint" "hellen-one-knock:knock"
+		(property "Footprint" "hellen-one-knock-0.2:knock"
 			(at 120.65 323.85 0)
 			(effects

Commit message: sync
Parts:
- J6: footprint Connector_Molex:Molex_Mini-Fit_Jr_5566-06A_2x03_P4.20mm_Vertical -> New_Connector_Molex:Molex_Mini-Fit_Jr_5566-06A_2x03_P4.20mm_Vertical
- J9: footprint Connector_Molex:Molex_Mini-Fit_Jr_5566-12A_2x06_P4.20mm_Vertical -> New_Connector_Molex:Molex_Mini-Fit_Jr_5566-12A_2x06_P4.20mm_Vertical
Connections:
- net 5V_OUT8 is gone; now on net 5V_OUT7: M1.W4 (IGN8)
- net +5VP: now also J7.10 (Pin_10), J7.12 (Pin_12), J7.14 (Pin_14), J7.16 (Pin_16); no longer J7.1 (Pin_1), J7.27 (Pin_27), J7.29 (Pin_29), J7.3 (Pin_3)
- net 5V_OUT1: now also J7.34 (Pin_34), M1.W10 (IGN2); no longer J1.106 (IGT), J7.31 (Pin_31), M1.W11 (IGN1)
- net 5V_OUT2: now also J7.32 (Pin_32), M1.W9 (IGN3); no longer J7.33 (Pin_33), M1.W10 (IGN2)
- net 5V_OUT3: now also J7.30 (Pin_30), M1.W8 (IGN4); no longer J7.35 (Pin_35), M1.W9 (IGN3)
- net 5V_OUT4: now also J7.28 (Pin_28), M1.W7 (IGN5); no longer J7.37 (Pin_37), M1.W8 (IGN4)
- net 5V_OUT5: now also J7.26 (Pin_26), M1.W6 (IGN6); no longer M1.W7 (IGN5)
- net 5V_OUT6: now also M1.W5 (IGN7); no longer M1.W6 (IGN6)
- net 5V_OUT7: no longer M1.W5 (IGN7)
- net AT1: now also J7.33 (Pin_33); no longer J7.13 (Pin_13)
- net AT2: now also J7.35 (Pin_35); no longer J7.15 (Pin_15)
- net AUX1: now also J7.23 (Pin_23); no longer J7.5 (Pin_5)
- net AUX2: now also J7.21 (Pin_21); no longer J7.7 (Pin_7)
- net AUX3: now also J7.19 (Pin_19); no longer J7.9 (Pin_9)
- net AUX4: now also J7.17 (Pin_17); no longer J7.11 (Pin_11)
- net D1_IN: now also J7.7 (Pin_7); no longer J7.25 (Pin_25)
- net D2_IN: now also J7.5 (Pin_5); no longer J7.23 (Pin_23)
- net D3_IN: now also J7.3 (Pin_3); no longer J7.21 (Pin_21)
- net D4_IN: now also J7.1 (Pin_1); no longer J7.19 (Pin_19)
- net DC Driver 1/PWM: now also M1.E28 (OUT_PWM8); no longer M1.E14 (OUT_PWM5)
- net DC1+: now also J9.7 (Pin_7); no longer J9.11 (Pin_11)
- net DC1-: now also J9.8 (Pin_8); no longer J9.12 (Pin_12)
- net GND: now also J7.6 (Pin_6), J7.8 (Pin_8); no longer J7.28 (Pin_28), J7.30 (Pin_30)
- net LS1_HOT_OUT: now also J1.125 (#20); no longer J1.112 (#10)
- net LS1_OUT: now also J9.9 (Pin_9); no longer J9.7 (Pin_7)
- net LS2_HOT_OUT: now also J1.112 (#10); no longer J1.125 (#20)
- net LS2_OUT: now also J9.10 (Pin_10); no longer J9.8 (Pin_8)
- net LS3_OUT: now also J9.11 (Pin_11); no longer J9.9 (Pin_9)
- net LS4_OUT: now also J9.12 (Pin_12); no longer J9.10 (Pin_10)
- net MAP2: now also J7.31 (Pin_31); no longer J7.6 (Pin_6)
- net MAP3: now also J7.29 (Pin_29); no longer J7.8 (Pin_8)
- net O2S2: now also J7.27 (Pin_27); no longer J7.16 (Pin_16)
- net PPS: now also J7.37 (Pin_37); no longer J7.10 (Pin_10)
- net PPS2: now also J7.40 (Pin_40); no longer J7.12 (Pin_12)
- net RES2: now also J7.25 (Pin_25); no longer J7.18 (Pin_18)
- net SENS1: now also J7.15 (Pin_15); no longer J7.26 (Pin_26)
- net SENS2: now also J7.13 (Pin_13); no longer J7.24 (Pin_24)
- net SENS3: now also J7.11 (Pin_11); no longer J7.22 (Pin_22)
- net SENS4: now also J7.9 (Pin_9); no longer J7.20 (Pin_20)
- net THRESH: now also M1.E14 (OUT_PWM5); no longer M1.E28 (OUT_PWM8)
- net TPS2: now also J7.39 (Pin_39); no longer J7.14 (Pin_14)
- net VRCAM+: now reaches J1.108 (I0F/G2)
- net VRCAM+: now also M3.W2 (VR+)
- net CAN1_HIGH renamed CAN1+
- net CAN1+: now also J7.22 (Pin_22); no longer J7.32 (Pin_32)
- net CAN1_LOW renamed CAN1-
- net CAN1-: now also J7.24 (Pin_24); no longer J7.34 (Pin_34)
- net CAN2_HIGH renamed CAN2+
- net CAN2+: now also J7.38 (Pin_38); no longer J7.36 (Pin_36)
- net CAN2_LOW renamed CAN2-
- net CAN2-: now also J7.36 (Pin_36); no longer J7.38 (Pin_38)
- net RES1: no longer names the net of M1.S17 (IN_RES1)
- net RES1: no longer J7.17 (Pin_17)
- net RES3: no longer names the net of M1.S18 (IN_RES3)
- net VREF1 renamed VREF_KNOCK
- new net SPARK: J1.106 (IGT), M1.W11 (IGN1)
- no-connect marks 28 -> 30
