File: EP91Starlet.kicad_sch (KiCad schematic)
At the start: 46 parts, among them J1 175446-6, J2 USB_B, J3 Conn_01x02, J5 Conn_01x02, J6 Conn_02x03_Top_Bottom, J7 Conn_02x20_Odd_Even, J9 Conn_02x06_Top_Bottom, M1 Module-mega-mcu144-0.7, M2 Module-vr-max9924-0.1, M3 Module-vr-discrete-0.5, M4 Module-power_12and5V-0.3, M5 Module-wbo-0.6, M6 Module-knock-0.2, M7 Module-can-0.1, Q2 BSS138, U1 VNLD5090-E, U2 VNLD5090-E, U3 VNLD5090-E, U4 VNLD5090-E, U5 VNLD5090-E, U6 VNLD5090-E

Commit message: sync
Connections:
- net +12V_RAW: now also J6.5 (Pin_5)
- net at M5.E1 (LSU_Un): now also J6.4 (Pin_4)
- net at M5.E2 (LSU_Vm): now also J6.6 (Pin_6)
- net at M5.E3 (LSU_Ip): now also J6.3 (Pin_3)
- net at M5.E4 (LSU_Rtrim): now also J6.1 (Pin_1)
- net at M5.E5 (LSU_Htr): now also J6.2 (Pin_2)
Other:
- moved on the sheet: J6
Changed lines of the file:
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@@
 	(wire
 		(pts
+			(xy 283.21 336.55) (xy 313.69 336.55)
+		)
+		(stroke
+			(width 0)
+			(type default)
+		)
+	)
+	(wire
+		(pts
 			(xy 55.88 34.29) (xy 66.04 34.29)
 		)
@@
 	(wire
 		(pts
+			(xy 313.69 336.55) (xy 313.69 327.66)
+		)
+		(stroke
+			(width 0)
+			(type default)
+		)
+	)
+	(wire
+		(pts
 			(xy 66.04 35.56) (xy 66.04 34.29)
 		)
@@
 	(wire
 		(pts
+			(xy 290.83 327.66) (xy 297.18 327.66)
+		)
+		(stroke
+			(width 0)
+			(type default)
+		)
+	)
+	(wire
+		(pts
 			(xy 68.58 194.31) (xy 78.74 194.31)
 		)
@@
 	(wire
 		(pts
+			(xy 284.48 335.28) (xy 284.48 334.01)
+		)
+		(stroke
+			(width 0)
+			(type default)
+		)
+	)
+	(wire
+		(pts
 			(xy 260.35 93.98) (xy 260.35 96.52)
 		)
@@
 	(wire
 		(pts
+			(xy 284.48 334.01) (xy 283.21 334.01)
+		)
+		(stroke
+			(width 0)
+			(type default)
+		)
+	)
+	(wire
+		(pts
 			(xy 72.39 101.6) (xy 71.12 101.6)
 		)
@@
 	(wire
 		(pts
+			(xy 283.21 328.93) (xy 290.83 328.93)
+		)
+		(stroke
+			(width 0)
+			(type default)
+		)
+	)
+	(wire
+		(pts
 			(xy 67.31 29.21) (xy 57.15 29.21)
 		)
@@
 	(wire
 		(pts
+			(xy 289.56 330.2) (xy 297.18 330.2)
+		)
+		(stroke
+			(width 0)
+			(type default)
+		)
+	)
+	(wire
+		(pts
+			(xy 309.88 335.28) (xy 309.88 332.74)
+		)
+		(stroke
+			(width 0)
+			(type default)
+		)
+	)
+	(wire
+		(pts
 			(xy 43.18 191.77) (xy 43.18 186.69)
 		)
@@
 	(wire
 		(pts
+			(xy 284.48 335.28) (xy 309.88 335.28)
+		)
+		(stroke
+			(width 0)
+			(type default)
+		)
+	)
+	(wire
+		(pts
 			(xy 71.12 106.68) (xy 81.28 106.68)
 		)
@@
 	(wire
 		(pts
+			(xy 290.83 331.47) (xy 290.83 332.74)
+		)
+		(stroke
+			(width 0)
+			(type default)
+		)
+	)
+	(wire
+		(pts
 			(xy 27.94 29.21) (xy 31.75 29.21)
 		)
@@
 	(wire
 		(pts
+			(xy 283.21 331.47) (xy 290.83 331.47)
+		)
+		(stroke
+			(width 0)
+			(type default)
+		)
+	)
+	(wire
+		(pts
 			(xy 30.48 144.78) (xy 46.99 144.78)
 		)
@@
 	(wire
 		(pts
+			(xy 313.69 327.66) (xy 309.88 327.66)
+		)
+		(stroke
+			(width 0)
+			(type default)
+		)
+	)
+	(wire
+		(pts
 			(xy 190.5 101.6) (xy 172.72 101.6)
 		)
@@
 	(wire
 		(pts
+			(xy 290.83 328.93) (xy 290.83 327.66)
+		)
+		(stroke
+			(width 0)
+			(type default)
+		)
+	)
+	(wire
+		(pts
 			(xy 81.28 146.05) (xy 81.28 144.78)
 		)
@@
 	(wire
 		(pts
+			(xy 283.21 326.39) (xy 289.56 326.39)
+		)
+		(stroke
+			(width 0)
+			(type default)
+		)
+	)
+	(wire
+		(pts
 			(xy 45.72 99.06) (xy 46.99 99.06)
 		)
@@
 	(wire
 		(pts
+			(xy 290.83 332.74) (xy 297.18 332.74)
+		)
+		(stroke
+			(width 0)
+			(type default)
+		)
+	)
+	(wire
+		(pts
 			(xy 81.28 336.55) (xy 78.74 336.55)
 		)
@@
 	(wire
 		(pts
+			(xy 289.56 326.39) (xy 289.56 330.2)
+		)
+		(stroke
+			(width 0)
+			(type default)
+		)
+	)
+	(wire
+		(pts
 			(xy 374.65 208.28) (xy 372.11 208.28)
 		)
@@
 	)
 	(symbol
+		(lib_id "hellen-one-common:+12V_RAW")
+		(at 309.88 330.2 270)
+		(unit 1)
+		(exclude_from_sim no)
+		(in_bom yes)
+		(on_board yes)
+		(dnp no)
+		(fields_autoplaced yes)
+		(property "Reference" "#PWR77"
+			(at 306.07 330.2 0)
+			(effects
+				(font
+					(size 1.27 1.27)
+				)
+				(hide yes)
+			)
+		)
+		(property "Value" "+12V_RAW"
+			(at 313.69 330.1999 90)
+			(effects
+				(font
+					(size 1.27 1.27)
+				)
+				(justify left)
+			)
+		)
+		(property "Footprint" ""
+			(at 309.88 330.2 0)
+			(effects
+				(font
+					(size 1.27 1.27)
+				)
+				(hide yes)
+			)
+		)
+		(property "Datasheet" ""
+			(at 309.88 330.2 0)
+			(effects
+				(font
+					(size 1.27 1.27)
+				)
+				(hide yes)
+			)
+		)
+		(property "Description" "Power symbol creates a global label with name \"+12V_RAW\""
+			(at 309.88 330.2 0)
+			(effects
+				(font
+					(size 1.27 1.27)
+				)
+				(hide yes)
+			)
+		)
+		(pin "1"
+		)
+		(instances
+			(project ""
+				(path "/10fbc709-889c-4565-8161-129ca9f0b73f"
+					(reference "#PWR77")
+					(unit 1)
+				)
+			)
+		)
+	)
+	(symbol
 		(lib_id "Device:R")
 		(at 101.6 30.48 270)
@@
 	(symbol
 		(lib_id "Connector_Generic:Conn_02x03_Top_Bottom")
-		(at 309.88 336.55 0)
+		(at 302.26 330.2 0)
 		(unit 1)
 		(exclude_from_sim no)
@@
 		(on_board yes)
 		(dnp no)
-		(fields_autoplaced yes)
 		(property "Reference" "J6"
-			(at 311.15 327.66 0)
+			(at 303.53 321.31 0)
 			(effects
 				(font
@@
 		)
 		(property "Value" "Conn_02x03_Top_Bottom"
-			(at 311.15 330.2 0)
+			(at 303.53 323.85 0)
 			(effects
 				(font
@@
 		)
 		(property "Footprint" "New_Connector_Molex:Molex_Mini-Fit_Jr_5566-06A_2x03_P4.20mm_Vertical"
-			(at 309.88 336.55 0)
+			(at 302.26 330.2 0)
 			(effects
 				(font
@@
 		)
 		(property "Datasheet" "~"
-			(at 309.88 336.55 0)
+			(at 302.26 330.2 0)
 			(effects
 				(font
@@
 		)
 		(property "Description" "Generic connector, double row, 02x03, top/bottom pin numbering scheme (row 1: 1...pins_per_row, row2: pins_per_row+1 ... num_pins), script generated (kicad-library-utils/schlib/autogen/connector/)"
-			(at 309.88 336.55 0)
+			(at 302.26 330.2 0)
 			(effects
 				(font

Commit message: sync
Connections:
- net CAN1+: now also J7.20 (Pin_20); no longer J7.22 (Pin_22)
- net CAN1-: now also J7.18 (Pin_18); no longer J7.24 (Pin_24)
Changed lines of the file:
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@@
-		)
-	)
-	(label "CAN1-"
-		(at 382.27 120.65 0)
-		(effects
-			(font
-				(size 1.27 1.27)
-			)
-			(justify left bottom)
 		)
 	)
@@
 		)
 	)
-	(label "CAN1+"
-		(at 382.27 118.11 0)
-		(effects
-			(font
-				(size 1.27 1.27)
-			)
-			(justify left bottom)
-		)
-	)
 	(label "VREF_KNOCK"
 		(at 189.23 241.3 180)
@@
 		)
 	)
+	(label "CAN1+"
+		(at 382.27 115.57 0)
+		(effects
+			(font
+				(size 1.27 1.27)
+			)
+			(justify left bottom)
+		)
+	)
 	(label "RES2"
 		(at 369.57 123.19 180)
@@
 		)
 	)
+	(label "CAN1-"
+		(at 382.27 113.03 0)
+		(effects
+			(font
+				(size 1.27 1.27)
+			)
+			(justify left bottom)
+		)
+	)
