File: EP91Starlet.kicad_sch (KiCad schematic)
At the start: 46 parts, among them IC1 VNLD5160-E, IC2 VNLD5160-E, IC3 VNLD5160-E, IC4 VNLD5160-E, IC5 VNLD5160-E, IC6 VNLD5160-E, J1 175446-6, J3 Conn_01x02, J4 USB_B_Mini, J5 Conn_01x02, J6 Conn_02x03_Top_Bottom, J7 Conn_02x20_Odd_Even, J9 Conn_02x06_Top_Bottom, M1 Module-mega-mcu144-0.7, M2 Module-vr-max9924-0.1, M3 Module-vr-discrete-0.5, M4 Module-power_12and5V-0.3, M5 Module-wbo-0.6, M6 Module-knock-0.2, M7 Module-can-0.1, Q2 BSS138

Commit message: sync
Connections:
- net CHECKENGINE_IN: now also M1.E8 (OUT_IO1); no longer M1.E12 (OUT_IO2)
- net DC Driver 1/DIR: now also M1.E13 (OUT_IO12); no longer M1.E6 (OUT_IO3)
- net DC Driver 1/DIS: now also M1.E20 (OUT_IO13); no longer M1.E7 (OUT_IO5)
- net DC Driver 1/PWM: now also M1.E26 (OUT_PWM6); no longer M1.E28 (OUT_PWM8)
- net FANRELAY_IN: now also M1.E6 (OUT_IO3); no longer M1.E21 (OUT_IO4)
- net FUELRELAY_IN: now also M1.E7 (OUT_IO5); no longer M1.E8 (OUT_IO1)
- net IACCLOSE_IN: now also M1.E16 (OUT_PWM3); no longer M1.E27 (OUT_PWM1)
- net IACOPEN_IN: now also M1.E15 (OUT_PWM4); no longer M1.E17 (OUT_PWM2)
Changed lines of the file:
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@@
 	(wire
 		(pts
-			(xy 170.18 106.68) (xy 170.18 93.98)
+			(xy 170.18 93.98) (xy 170.18 127)
 		)
 		(stroke
@@
 	(wire
 		(pts
+			(xy 165.1 88.9) (xy 168.91 88.9)
+		)
+		(stroke
+			(width 0)
+			(type default)
+		)
+	)
+	(wire
+		(pts
 			(xy 68.58 194.31) (xy 78.74 194.31)
 		)
@@
 	(wire
 		(pts
+			(xy 168.91 88.9) (xy 168.91 83.82)
+		)
+		(stroke
+			(width 0)
+			(type default)
+		)
+	)
+	(wire
+		(pts
+			(xy 172.72 91.44) (xy 172.72 124.46)
+		)
+		(stroke
+			(width 0)
+			(type default)
+		)
+	)
+	(wire
+		(pts
 			(xy 105.41 30.48) (xy 106.68 30.48)
 		)
@@
 	(wire
 		(pts
-			(xy 172.72 101.6) (xy 172.72 91.44)
-		)
-		(stroke
-			(width 0)
-			(type default)
-		)
-	)
-	(wire
-		(pts
 			(xy 68.58 231.14) (xy 78.74 231.14)
 		)
@@
 	(wire
 		(pts
+			(xy 170.18 127) (xy 190.5 127)
+		)
+		(stroke
+			(width 0)
+			(type default)
+		)
+	)
+	(wire
+		(pts
 			(xy 382.27 105.41) (xy 382.27 107.95)
 		)
@@
 	(wire
 		(pts
-			(xy 190.5 101.6) (xy 172.72 101.6)
-		)
-		(stroke
-			(width 0)
-			(type default)
-		)
-	)
-	(wire
-		(pts
 			(xy 147.32 88.9) (xy 146.05 88.9)
 		)
@@
 	(wire
 		(pts
+			(xy 168.91 83.82) (xy 190.5 83.82)
+		)
+		(stroke
+			(width 0)
+			(type default)
+		)
+	)
+	(wire
+		(pts
 			(xy 40.64 137.16) (xy 40.64 144.78)
 		)
@@
 	(wire
 		(pts
-			(xy 165.1 88.9) (xy 190.5 88.9)
-		)
-		(stroke
-			(width 0)
-			(type default)
-		)
-	)
-	(wire
-		(pts
 			(xy 30.48 72.39) (xy 30.48 60.96)
 		)
@@
 	(wire
 		(pts
-			(xy 190.5 106.68) (xy 170.18 106.68)
-		)
-		(stroke
-			(width 0)
-			(type default)
-		)
-	)
-	(wire
-		(pts
 			(xy 69.85 226.06) (xy 69.85 232.41)
 		)
@@
 		(pts
 			(xy 80.01 231.14) (xy 78.74 231.14)
+		)
+		(stroke
+			(width 0)
+			(type default)
+		)
+	)
+	(wire
+		(pts
+			(xy 172.72 124.46) (xy 190.5 124.46)
 		)
 		(stroke
@@
 		)
 	)
+	(label "CHECKENGINE_IN"
+		(at 190.5 96.52 180)
+		(effects
+			(font
+				(size 1.27 1.27)
+			)
+			(justify right bottom)
+		)
+	)
 	(label "5V_OUT7"
 		(at 190.5 38.1 180)
@@
 		)
 	)
+	(label "FANRELAY_IN"
+		(at 190.5 101.6 180)
+		(effects
+			(font
+				(size 1.27 1.27)
+			)
+			(justify right bottom)
+		)
+	)
 	(label "VIGN"
 		(at 190.5 254 180)
@@
 		)
 	)
-	(label "IACOPEN_IN"
-		(at 190.5 73.66 180)
-		(effects
-			(font
-				(size 1.27 1.27)
-			)
-			(justify right bottom)
-		)
-	)
 	(label "LS4_HOT_OUT"
 		(at 27.94 58.42 180)
@@
 		)
 	)
-	(label "FANRELAY_IN"
-		(at 190.5 104.14 180)
+	(label "FUELRELAY_IN"
+		(at 190.5 106.68 180)
 		(effects
 			(font
@@
 		)
 	)
-	(label "FUELRELAY_IN"
-		(at 190.5 96.52 180)
-		(effects
-			(font
-				(size 1.27 1.27)
-			)
-			(justify right bottom)
-		)
-	)
 	(label "AT2"
 		(at 369.57 135.89 180)
@@
 		)
 	)
-	(label "CHECKENGINE_IN"
-		(at 190.5 99.06 180)
-		(effects
-			(font
-				(size 1.27 1.27)
-			)
-			(justify right bottom)
-		)
-	)
 	(label "CAN1+"
 		(at 382.27 113.03 0)
@@
 		)
 	)
-	(label "IACCLOSE_IN"
-		(at 190.5 71.12 180)
-		(effects
-			(font
-				(size 1.27 1.27)
-			)
-			(justify right bottom)
-		)
-	)
 	(label "DC1+"
 		(at 147.32 91.44 180)
@@
 		)
 	)
+	(label "IACOPEN_IN"
+		(at 190.5 78.74 180)
+		(effects
+			(font
+				(size 1.27 1.27)
+			)
+			(justify right bottom)
+		)
+	)
 	(label "LS2_IN"
 		(at 190.5 58.42 180)
@@
 		(effects
 			(font
+				(size 1.27 1.27)
+			)
+			(justify right bottom)
+		)
+	)
+	(label "IACCLOSE_IN"
+		(at 190.5 76.2 180)
+		(effects
+			(font
