File: _autosave-EP91Starlet.kicad_sch (KiCad schematic)
At the start: 42 parts, among them J1 175446-6, J2 Extra Inputs (2.54mm Pin Head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, J3 TE_6473423-1_26p, M1 Module-mega-mcu144-0.7, M2 Module-vr-max9924-0.1, M3 Module-vr-discrete-0.5, M4 Module-power_12and5V-0.3, M5 Module-wbo-0.6, M6 Module-knock-0.2, M7 Module-can-0.1, Q2 BSS138, U1 VNLD5090-E, U2 VNLD5090-E, U3 VNLD5090-E, U4 VNLD5090-E, U5 VNLD5090-E, U6 VNLD5090-E

Commit message: sync
Changed lines of the file:
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@@
-	)
-	(symbol
-		(lib_id "Connectors:TE_6473423-1_26p")
-		(at 298.45 130.81 0)
-		(unit 1)
-		(exclude_from_sim no)
-		(in_bom yes)
-		(on_board yes)
-		(dnp no)
-		(fields_autoplaced yes)
-		(property "Reference" "J3"
-			(at 295.91 124.46 0)
-			(effects
-				(font
-					(size 1.27 1.27)
-				)
-			)
-		)
-		(property "Value" "TE_6473423-1_26p"
-			(at 295.91 127 0)
-			(effects
-				(font
-					(size 1.27 1.27)
-				)
-			)
-		)
-		(property "Footprint" "TE:6473423-1"
-			(at 302.26 200.025 0)
-			(effects
-				(font
-					(size 1.27 1.27)
-				)
-				(hide yes)
-			)
-		)
-		(property "Datasheet" ""
-			(at 298.45 125.095 0)
-			(effects
-				(font
-					(size 1.27 1.27)
-				)
-				(hide yes)
-			)
-		)
-		(property "Description" "26 pin connector"
-			(at 298.45 130.81 0)
-			(effects
-				(font
-					(size 1.27 1.27)
-				)
-				(hide yes)
-			)
-		)
-		(pin "9"
-		)
-		(pin "20"
-		)
-		(pin "23"
-		)
-		(pin "11"
-		)
-		(pin "7"
-		)
-		(pin "25"
-		)
-		(pin "10"
-		)
-		(pin "13"
-		)
-		(pin "18"
-		)
-		(pin "12"
-		)
-		(pin "21"
-		)
-		(pin "24"
-		)
-		(pin "17"
-		)
-		(pin "15"
-		)
-		(pin "14"
-		)
-		(pin "8"
-		)
-		(pin "16"
-		)
-		(pin "6"
-		)
-		(pin "5"
-		)
-		(pin "3"
-		)
-		(pin "2"
-		)
-		(pin "4"
-		)
-		(pin "26"
-		)
-		(pin "19"
-		)
-		(pin "22"
-		)
-		(pin "1"
-		)
-		(instances
-			(project ""
-				(path "/10fbc709-889c-4565-8161-129ca9f0b73f"
-					(reference "J3")
-					(unit 1)
-				)
-			)
-		)
 	)
 	(symbol
@@
 					(unit 1)
 				)
+			)
+		)
+	)
+	(symbol
+		(lib_id "Connectors:TE_6473423-1_26p")
+		(at 295.91 129.54 0)
+		(unit 1)
+		(exclude_from_sim no)
+		(in_bom yes)
+		(on_board yes)
+		(dnp no)
+		(fields_autoplaced yes)
+		(property "Reference" "J3"
+			(at 293.37 123.19 0)
+			(effects
+				(font
+					(size 1.27 1.27)
+				)
+			)
+		)
+		(property "Value" "TE_6473423-1_26p"
+			(at 293.37 125.73 0)
+			(effects
+				(font
+					(size 1.27 1.27)
+				)
+			)
+		)
+		(property "Footprint" "TE:6473423-1"
+			(at 299.72 198.755 0)
+			(effects
+				(font
+					(size 1.27 1.27)
+				)
+				(hide yes)
+			)
+		)
+		(property "Datasheet" ""
+			(at 295.91 123.825 0)
+			(effects
+				(font
+					(size 1.27 1.27)
+				)
+				(hide yes)
+			)
+		)
+		(property "Description" "26 pin connector"
+			(at 295.91 129.54 0)
+			(effects
+				(font
+					(size 1.27 1.27)
+				)
+				(hide yes)
+			)
+		)
+		(pin "22"
+		)
+		(pin "11"
+		)
+		(pin "16"
+		)
+		(pin "17"
+		)
+		(pin "18"
+		)
+		(pin "13"
+		)
+		(pin "9"
+		)
+		(pin "1"
+		)
+		(pin "6"
+		)
+		(pin "4"
+		)
+		(pin "7"
+		)
+		(pin "24"
+		)
+		(pin "20"
+		)
+		(pin "21"
+		)
+		(pin "15"
+		)
+		(pin "12"
+		)
+		(pin "5"
+		)
+		(pin "14"
+		)
+		(pin "23"
+		)
+		(pin "19"
+		)
+		(pin "26"
+		)
+		(pin "25"
+		)
+		(pin "2"
+		)
+		(pin "3"
+		)
+		(pin "8"
+		)
+		(pin "10"
+		)
+		(instances
+			(project ""
+				(path "/10fbc709-889c-4565-8161-129ca9f0b73f"
+					(reference "J3")
+					(unit 1)
+				)
