File: DC_MOTOR_0.1.kicad_sch (KiCad schematic)
At the start: 17 parts, among them P1 Pad, P2 Pad, U8 TLE9201SG

Commit message: sync
Parts:
- removed P1, P2: Pad, hellen-one-common:PAD-TH, symbol hellen-one-common:Pad
- C10, C11, C12, C13, C14, C15, C6, C7, C8, C9: footprint hellen-one-common:C0805 -> Capacitor_SMD:C_0603_1608Metric
- C16, C17, C18: footprint hellen-one-common:C0603 -> Capacitor_SMD:C_0603_1608Metric
- R15: footprint hellen-one-common:R0603 -> Resistor_SMD:R_0603_1608Metric
Changed lines of the file:
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@@
-	)
-	(junction
-		(at 207.01 95.25)
-		(diameter 0)
-		(color 0 0 0 0)
 	)
 	(junction
@@
 	)
 	(junction
-		(at 207.01 97.79)
-		(diameter 0)
-		(color 0 0 0 0)
-	)
-	(junction
 		(at 91.44 71.12)
 		(diameter 0)
@@
 	(wire
 		(pts
-			(xy 207.01 95.25) (xy 218.44 95.25)
-		)
-		(stroke
-			(width 0)
-			(type default)
-		)
-	)
-	(wire
-		(pts
 			(xy 166.37 92.71) (xy 166.37 87.63)
 		)
@@
 	(wire
 		(pts
-			(xy 194.31 95.25) (xy 207.01 95.25)
-		)
-		(stroke
-			(width 0)
-			(type default)
-		)
-	)
-	(wire
-		(pts
-			(xy 207.01 97.79) (xy 207.01 99.06)
+			(xy 194.31 95.25) (xy 218.44 95.25)
 		)
 		(stroke
@@
 	(wire
 		(pts
-			(xy 207.01 97.79) (xy 218.44 97.79)
-		)
-		(stroke
-			(width 0)
-			(type default)
-		)
-	)
-	(wire
-		(pts
 			(xy 210.82 92.71) (xy 218.44 92.71)
 		)
@@
 	(wire
 		(pts
-			(xy 207.01 95.25) (xy 207.01 96.52)
-		)
-		(stroke
-			(width 0)
-			(type default)
-		)
-	)
-	(wire
-		(pts
 			(xy 100.33 71.12) (xy 109.22 71.12)
 		)
@@
 	(wire
 		(pts
-			(xy 194.31 97.79) (xy 207.01 97.79)
+			(xy 194.31 97.79) (xy 218.44 97.79)
 		)
 		(stroke
@@
 			)
 		)
-		(property "Footprint" "hellen-one-common:C0805"
+		(property "Footprint" "Capacitor_SMD:C_0603_1608Metric"
 			(at 77.47 77.47 0)
 			(effects
@@
 			)
 		)
-		(property "Footprint" "hellen-one-common:C0805"
+		(property "Footprint" "Capacitor_SMD:C_0603_1608Metric"
 			(at 86.36 77.47 0)
 			(effects
@@
 	)
 	(symbol
-		(lib_id "hellen-one-common:Pad")
-		(at 212.09 99.06 0)
-		(unit 1)
-		(exclude_from_sim no)
-		(in_bom yes)
-		(on_board yes)
-		(dnp no)
-		(property "Reference" "P2"
-			(at 213.36 99.06 0)
-			(effects
-				(font
-					(size 1.27 1.27)
-				)
-				(justify left)
-			)
-		)
-		(property "Value" "Pad"
-			(at 212.09 101.6 0)
-			(effects
-				(font
-					(size 1.27 1.27)
-				)
-				(hide yes)
-			)
-		)
-		(property "Footprint" "hellen-one-common:PAD-TH"
-			(at 212.09 102.87 0)
-			(effects
-				(font
-					(size 1.27 1.27)
-				)
-				(hide yes)
-			)
-		)
-		(property "Datasheet" "~"
-			(at 212.09 99.06 0)
-			(effects
-				(font
-					(size 1.27 1.27)
-				)
-				(hide yes)
-			)
-		)
-		(property "Description" ""
-			(at 212.09 99.06 0)
-			(effects
-				(font
-					(size 1.27 1.27)
-				)
-				(hide yes)
-			)
-		)
-		(pin "1"
-		)
-		(instances
-			(project "EP91Starlet"
-				(path "/10fbc709-889c-4565-8161-129ca9f0b73f/a3a2cbd2-512c-466e-b8f9-d557249ac1e6"
-					(reference "P2")
-					(unit 1)
-				)
-			)
-		)
-	)
-	(symbol
 		(lib_id "power:GND")
 		(at 166.37 106.68 0)
@@
 	)
 	(symbol
-		(lib_id "hellen-one-common:Pad")
-		(at 212.09 96.52 0)
-		(unit 1)
-		(exclude_from_sim no)
-		(in_bom yes)
-		(on_board yes)
-		(dnp no)
-		(property "Reference" "P1"
-			(at 213.36 96.52 0)
-			(effects
-				(font
-					(size 1.27 1.27)
-				)
-				(justify left)
-			)
-		)
-		(property "Value" "Pad"
-			(at 212.09 99.06 0)
-			(effects
-				(font
-					(size 1.27 1.27)
-				)
-				(hide yes)
-			)
-		)
-		(property "Footprint" "hellen-one-common:PAD-TH"
-			(at 212.09 100.33 0)
-			(effects
-				(font
-					(size 1.27 1.27)
-				)
-				(hide yes)
-			)
-		)
-		(property "Datasheet" "~"
-			(at 212.09 96.52 0)
-			(effects
-				(font
-					(size 1.27 1.27)
-				)
-				(hide yes)
-			)
-		)
-		(property "Description" ""
-			(at 212.09 96.52 0)
-			(effects
-				(font
-					(size 1.27 1.27)
-				)
-				(hide yes)
-			)
-		)
-		(pin "1"
-		)
-		(instances
-			(project "EP91Starlet"
-				(path "/10fbc709-889c-4565-8161-129ca9f0b73f/a3a2cbd2-512c-466e-b8f9-d557249ac1e6"
-					(reference "P1")
-					(unit 1)
-				)
-			)
-		)
-	)
-	(symbol
 		(lib_id "hellen-one-common:Cap")
 		(at 153.67 74.93 90)
@@
 			)
 		)
-		(property "Footprint" "hellen-one-common:C0603"
+		(property "Footprint" "Capacitor_SMD:C_0603_1608Metric"
 			(at 157.48 77.47 0)
 			(effects
@@
 			)
 		)
-		(property "Footprint" "hellen-one-common:C0805"
+		(property "Footprint" "Capacitor_SMD:C_0603_1608Metric"
 			(at 68.58 77.47 0)
 			(effects
@@
 			)
 		)
-		(property "Footprint" "hellen-one-common:C0603"
+		(property "Footprint" "Capacitor_SMD:C_0603_1608Metric"
 			(at 170.18 105.41 0)
 			(effects
@@
 			)
 		)
-		(property "Footprint" "hellen-one-common:C0805"
+		(property "Footprint" "Capacitor_SMD:C_0603_1608Metric"
 			(at 104.14 77.47 0)
 			(effects
@@
 			)
 		)
-		(property "Footprint" "hellen-one-common:C0805"
+		(property "Footprint" "Capacitor_SMD:C_0603_1608Metric"
 			(at 139.7 77.47 0)
 			(effects
@@
 			)
 		)
-		(property "Footprint" "hellen-one-common:C0805"
+		(property "Footprint" "Capacitor_SMD:C_0603_1608Metric"
 			(at 113.03 77.47 0)
 			(effects
@@
 			)
 		)
-		(property "Footprint" "hellen-one-common:C0603"
+		(property "Footprint" "Capacitor_SMD:C_0603_1608Metric"
 			(at 170.18 81.28 0)
 			(effects
@@
 			)
 		)
-		(property "Footprint" "hellen-one-common:C0805"
+		(property "Footprint" "Capacitor_SMD:C_0603_1608Metric"
 			(at 121.92 77.47 0)
 			(effects
@@
 			)
 		)
-		(property "Footprint" "hellen-one-common:C0805"
+		(property "Footprint" "Capacitor_SMD:C_0603_1608Metric"
 			(at 130.81 77.47 0)
 			(effects
@@
 			)
 		)
-		(property "Footprint" "hellen-one-common:R0603"
+		(property "Footprint" "Resistor_SMD:R_0603_1608Metric"
 			(at 214.63 86.36 0)
 			(effects
@@
 			)
 		)
-		(property "Footprint" "hellen-one-common:C0805"
+		(property "Footprint" "Capacitor_SMD:C_0603_1608Metric"
 			(at 148.59 77.47 0)
 			(effects
@@
 			)
 		)
-		(property "Footprint" "hellen-one-common:C0805"
+		(property "Footprint" "Capacitor_SMD:C_0603_1608Metric"
 			(at 95.25 77.47 0)
 			(effects
