File: EGT.kicad_sch (KiCad schematic)
At the start: 9 parts, among them U7 MAX31855KASA

Commit message: sync
Parts:
- C1, C2, C3, C4, C5: footprint hellen-one-common:C0603 -> Capacitor_SMD:C_0603_1608Metric
Changed lines of the file:
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@@
 			)
 		)
-		(property "Footprint" "hellen-one-common:C0603"
+		(property "Footprint" "Capacitor_SMD:C_0603_1608Metric"
 			(at 191.77 78.74 0)
 			(effects
@@
 			)
 		)
-		(property "Footprint" "hellen-one-common:C0603"
+		(property "Footprint" "Capacitor_SMD:C_0603_1608Metric"
 			(at 179.07 78.74 0)
 			(effects
@@
 			)
 		)
-		(property "Footprint" "hellen-one-common:C0603"
+		(property "Footprint" "Capacitor_SMD:C_0603_1608Metric"
 			(at 144.78 96.52 0)
 			(effects
@@
 			)
 		)
-		(property "Footprint" "hellen-one-common:C0603"
+		(property "Footprint" "Capacitor_SMD:C_0603_1608Metric"
 			(at 138.43 106.68 0)
 			(effects
@@
 			)
 		)
-		(property "Footprint" "hellen-one-common:C0603"
+		(property "Footprint" "Capacitor_SMD:C_0603_1608Metric"
 			(at 153.67 106.68 0)
 			(effects
