File: EP91Starlet.kicad_pcb (KiCad board)
At the start: 4 copper layers, 100 x 100 mm, 46 parts, among them J1 Conn_02x04_Top_Bottom, J2 Conn_02x03_Top_Bottom, J3 Conn_02x10_Top_Bottom, J4 Conn_02x03_Odd_Even, J5 USB_B, J6 Conn_02x04_Top_Bottom, J7 Conn_02x03_Odd_Even, J8 Conn_01x02, M1 Module-vr-max9924-0.1, M2 Module-mega-mcu144-0.7, M3 Module-knock-0.2, M4 Module-wbo-0.5, M5 Module-vr-max9924-0.1, M6 Module-power_12and5V-0.3, M7 Module-can-0.1, U1 VNLD5160TR-E, U2 VNLD5160TR-E, U3 VNLD5160TR-E, U4 VNLD5160TR-E, U5 VNLD5160TR-E, U6 VNLD5160TR-E

Commit message: retry (last time i promise :))
Parts:
- removed D1, D2, D3, D4, D5, D6, D7, D8: B5819W, footprints:SOD-123
- removed J1, J6: Conn_02x04_Top_Bottom, Connector_Molex:Molex_Mini-Fit_Jr_5569-08A2_2x04_P4.20mm_Horizontal
- removed J2: Conn_02x03_Top_Bottom, Connector_Molex:Molex_Mini-Fit_Jr_5569-06A2_2x03_P4.20mm_Horizontal
- removed J3: Conn_02x10_Top_Bottom, Connector_Molex:Molex_Mini-Fit_Jr_5569-20A2_2x10_P4.20mm_Horizontal
- removed J4, J7: Conn_02x03_Odd_Even, Connector_PinHeader_2.54mm:PinHeader_2x03_P2.54mm_Vertical
- removed J5: USB_B, footprints:USB_B
- removed J8: Conn_01x02, Connector_PinHeader_2.54mm:PinHeader_2x01_P2.54mm_Vertical
- removed M1, M5: Module-vr-max9924-0.1, vrmax9924:vr-max9924
- removed M2: Module-mega-mcu144-0.7, megamcu144:mega-mcu144
- removed M3: Module-knock-0.2, knock:knock
- removed M4: Module-wbo-0.5, wbo:wbo
- removed M6: Module-power_12and5V-0.3, power5_12:power_12and5V
- removed M7: Module-can-0.1, can:can
- removed R1, R17, R18, R19, R2, R20, R3, R4, R5, R6, R7, R8: 4.7k, footprints:R0603
- removed REF** (x4): MountingHole_3.2mm_M3_Pad_Via, MountingHole:MountingHole_3.2mm_M3_Pad_Via
- removed U1, U2, U3, U4, U5, U6: VNLD5160TR-E, Package_SO:SOIC-8_3.9x4.9mm_P1.27mm
- removed U7: ~, ul_175446-6:CONN_175446-6_TYCO_TYC
Routing:
- net +12V_RAW: track 222.7 -> 0.00 mm, vias 6 -> 0
- net +5VP: track 159.8 -> 0.00 mm
- net Net-(J1-Pin_4): track 116.5 -> 0.00 mm
- net +5VA: track 116.5 -> 0.00 mm
- net Net-(J1-Pin_3): track 111.3 -> 0.00 mm
- net Net-(J1-Pin_2): track 111.0 -> 0.00 mm
- net Net-(J1-Pin_1): track 110.1 -> 0.00 mm
- net Net-(J3-Pin_10): track 88.3 -> 0.00 mm
- net Net-(J3-Pin_9): track 78.0 -> 0.00 mm
- net Net-(J3-Pin_8): track 71.6 -> 0.00 mm
- net /LS_PROTECTED_2 C/IN1: track 69.6 -> 0.00 mm, vias 2 -> 0
- net Net-(M6-V12_PERM): track 68.5 -> 0.00 mm
- net /INJ4/OUT2: track 67.9 -> 0.00 mm
- net Net-(M2-IN_D1): track 66.4 -> 0.00 mm, vias 1 -> 0
- net /LS_PROTECTED_2 C/IN2: track 65.9 -> 0.00 mm, vias 2 -> 0
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- removed copper zone on B.Cu, net GND
- removed copper zone on F.Cu, net GND
- removed copper zone on In1.Cu, net GND
- removed copper zone on In2.Cu, net GND
Other:
- board outline removed

Commit message: sync
Parts:
- added J1: 175446-6, 175446-6:1754466, F.Cu at (89.2, 27.7)

Commit message: sync
Parts:
- added J2: Conn_02x15_Top_Bottom, Connector_PinHeader_2.54mm:PinHeader_2x15_P2.54mm_Vertical, F.Cu at (141.9, 116.5)
- added M1: Module-mega-mcu144-0.7, mega-mcu144:mega-mcu144, F.Cu at (96.8, 88.7)
- added M2: Module-vr-max9924-0.1, vr-max9924:vr-max9924, F.Cu at (140.4, 58.4)
- added M3: Module-vr-discrete-0.5, vr-discrete:vr-discrete, F.Cu at (140.4, 69.4)
- added M4: Module-power_12and5V-0.3, power_12and5V:power_12and5V, F.Cu at (125.8, 110.8)
- added M5: Module-wbo-0.5, wbo:wbo, F.Cu at (96.8, 104.0)
- moved J1 11.8 mm to (94.0, 38.5)
Connections:
- J1 pad 10: unconnected-(J1-Pad10) -> /CHECKENGINELIGHT
- J1 pad 101: unconnected-(J1-Pad101) -> /IACCLOSE
- J1 pad 103: unconnected-(J1-Pad103) -> /COOLANT
- J1 pad 104: unconnected-(J1-Pad104) -> /MAP
- J1 pad 105: unconnected-(J1-Pad105) -> /AIR
- J1 pad 106: unconnected-(J1-Pad106) -> /SPARK1
- J1 pad 109: unconnected-(J1-Pad109) -> /VR-
- J1 pad 11: unconnected-(J1-Pad11) -> /CATCONVERTLIGHT
- J1 pad 110: unconnected-(J1-Pad110) -> /O2SENS
- J1 pad 112: unconnected-(J1-Pad112) -> /INJ1
- J1 pad 113: unconnected-(J1-Pad113) -> GND
- J1 pad 114: unconnected-(J1-Pad114) -> /IACOPEN
- J1 pad 115: unconnected-(J1-Pad115) -> /O2HEAT
- J1 pad 116: unconnected-(J1-Pad116) -> GNDA
- J1 pad 117: unconnected-(J1-Pad117) -> /TPS
- J1 pad 118: unconnected-(J1-Pad118) -> +5VP
- J1 pad 119: unconnected-(J1-Pad119) -> /IDLESWITCH
- J1 pad 121: unconnected-(J1-Pad121) -> /VRCRANK+
- J1 pad 124: unconnected-(J1-Pad124) -> GND
- J1 pad 125: unconnected-(J1-Pad125) -> /INJ2
- J1 pad 2: unconnected-(J1-Pad2) -> +12V_PERM
- J1 pad 9: unconnected-(J1-Pad9) -> +12V_RAW
- J1 pad MH1: unconnected-(J1-PadMH1) -> GND
- J1 pad MH2: unconnected-(J1-PadMH2) -> GND
- J1 pad MH3: unconnected-(J1-PadMH3) -> GND

Commit message: sync
Parts:
- added D1: B5819W, Diode_SMD:D_SOD-123, F.Cu at (63.2, 83.6)
- added D2: B5819W, Diode_SMD:D_SOD-123, F.Cu at (63.2, 87.0)
- added D3: B5819W, Diode_SMD:D_SOD-123, F.Cu at (63.2, 90.3)
- added D4: B5819W, Diode_SMD:D_SOD-123, F.Cu at (63.2, 93.7)
- added D5: 1N4148WS, Diode_SMD:D_SOD-323, F.Cu at (99.0, 93.4)
- added D6: B5819W, Diode_SMD:D_SOD-123, F.Cu at (63.2, 97.0)
- added D7: B5819W, Diode_SMD:D_SOD-123, F.Cu at (63.2, 100.4)
- added D8: B5819W, Diode_SMD:D_SOD-123, F.Cu at (63.2, 103.7)
- added D9: B5819W, Diode_SMD:D_SOD-123, F.Cu at (63.2, 107.1)
- added M6: Module-knock-0.2, knock:knock, F.Cu at (87.5, 70.1)
- added Q2: BSS138, Package_TO_SOT_SMD:SOT-23, F.Cu at (94.3, 94.3)
- added R1: 4.7k, Resistor_SMD:R_0402_1005Metric, F.Cu at (93.4, 82.9)
- added R10: 510R, Resistor_SMD:R_0402_1005Metric, F.Cu at (96.3, 90.9)
- added R11: 4.7k, Resistor_SMD:R_0402_1005Metric, F.Cu at (99.2, 82.9)
- added R12: 4.7k, Resistor_SMD:R_0402_1005Metric, F.Cu at (99.2, 84.9)
- added R13: 4.7k, Resistor_SMD:R_0402_1005Metric, F.Cu at (99.2, 86.9)
- added R14: 4.7k, Resistor_SMD:R_0402_1005Metric, F.Cu at (99.2, 88.9)
- added R2: 4.7k, Resistor_SMD:R_0402_1005Metric, F.Cu at (93.4, 84.9)
- added R3: 4.7k, Resistor_SMD:R_0402_1005Metric, F.Cu at (93.4, 86.9)
- added R4: 4.7k, Resistor_SMD:R_0402_1005Metric, F.Cu at (93.4, 88.9)
- added R5: 4.7k, Resistor_SMD:R_0402_1005Metric, F.Cu at (93.4, 90.9)
- added R6: 4.7k, Resistor_SMD:R_0402_1005Metric, F.Cu at (96.3, 82.9)
- added R7: 4.7k, Resistor_SMD:R_0402_1005Metric, F.Cu at (96.3, 84.9)
- added R8: 4.7k, Resistor_SMD:R_0402_1005Metric, F.Cu at (96.3, 86.9)
- added R9: 10k, Resistor_SMD:R_0402_1005Metric, F.Cu at (96.3, 88.9)
- added U1: VNLD5090-E, VNLD5090-E:VNLD5090-E, F.Cu at (113.0, 84.2)
- added U2: VNLD5090-E, VNLD5090-E:VNLD5090-E, F.Cu at (113.0, 77.6)
- added U3: VNLD5090-E, VNLD5090-E:VNLD5090-E, F.Cu at (167.0, 60.0)
- added U4: VNLD5090-E, VNLD5090-E:VNLD5090-E, F.Cu at (173.0, 60.0)
- added U5: VNLD5090-E, VNLD5090-E:VNLD5090-E, F.Cu at (185.4, 116.0)
- added U6: VNLD5090-E, VNLD5090-E:VNLD5090-E, F.Cu at (192.0, 116.0)
- M5: value Module-wbo-0.5 -> Module-wbo-0.6
- moved M5 122.0 mm to (218.6, 98.3), turned to 90 degrees
- moved M1 85.8 mm to (180.5, 70.1), turned to 180 degrees
- moved M3 63.2 mm to (203.3, 75.0), turned to 90 degrees
- moved M2 55.4 mm to (193.2, 75.1), turned to 90 degrees
- moved J1 52.8 mm to (144.4, 54.0)
- moved M4 25.6 mm to (135.0, 134.6)
- moved J2 20.1 mm to (160.3, 124.5), turned to 90 degrees
Connections:
- net /IN_CAM renamed /CAM
- net /IN_CRANK renamed /CRANK
- net /O2HEAT renamed /O2HEAT_OUT
- J1 pad 10: /CHECKENGINELIGHT -> /CHECKENGINE_OUT
- J1 pad 101: /IACCLOSE -> /IACCLOSE_OUT
- J1 pad 11: /CATCONVERTLIGHT -> unconnected-(J1-EGW-Pad11)
- J1 pad 114: /IACOPEN -> /IACOPEN_OUT
- J1 pad 120: unconnected-(J1-FAN-Pad120) -> /FANRELAY_OUT
- J1 pad 13: unconnected-(J1-SPD-Pad13) -> /VSS
- J1 pad 4: unconnected-(J1-FC-Pad4) -> /FUELRELAY_OUT
- J2 pad 1: unconnected-(J2-Pin_1-Pad1) -> /LS4_OUT
- J2 pad 2: unconnected-(J2-Pin_2-Pad2) -> /LS3_OUT
- J2 pad 3: unconnected-(J2-Pin_3-Pad3) -> /LS2_OUT
- J2 pad 4: unconnected-(J2-Pin_4-Pad4) -> /LS1_OUT
- J2 pad 5: unconnected-(J2-Pin_5-Pad5) -> /D1_IN
- J2 pad 6: unconnected-(J2-Pin_6-Pad6) -> /D2_IN
- J2 pad 7: unconnected-(J2-Pin_7-Pad7) -> /D3_IN
- J2 pad 8: unconnected-(J2-Pin_8-Pad8) -> /D4_IN
- J2 pad 9: unconnected-(J2-Pin_9-Pad9) -> /KNOCK_RAW
- M1 pad E12: unconnected-(M1-OUT_IO2-PadE12) -> /CHECKENGINE_IN
- M1 pad E14: unconnected-(M1-OUT_PWM5-PadE14) -> /LS3_IN
- M1 pad E15: unconnected-(M1-OUT_PWM4-PadE15) -> /LS2_IN
- M1 pad E16: unconnected-(M1-OUT_PWM3-PadE16) -> /LS1_IN
- M1 pad E17: unconnected-(M1-OUT_PWM2-PadE17) -> /IACOPEN_IN
- M1 pad E21: unconnected-(M1-OUT_IO4-PadE21) -> /FANRELAY_IN
- M1 pad E26: unconnected-(M1-OUT_PWM6-PadE26) -> /LS4_IN
- M1 pad E27: unconnected-(M1-OUT_PWM1-PadE27) -> /IACCLOSE_IN
- M1 pad E28: unconnected-(M1-OUT_PWM8-PadE28) -> /THRESH
- M1 pad E38: unconnected-(M1-V5A_SWITCHABLE-PadE38) -> +5VA
- M1 pad E39: unconnected-(M1-GNDA-PadE39) -> GNDA
- M1 pad E6: unconnected-(M1-OUT_IO3-PadE6) -> /CHECKCAT_IN
- M1 pad E8: unconnected-(M1-OUT_IO1-PadE8) -> /FUELRELAY_IN
- M1 pad G: unconnected-(M1-GND-PadG) -> GND
- M1 pad N22: unconnected-(M1-V33-PadN22) -> +3.3V
- M1 pad N26: unconnected-(M1-IN_VIGN-PadN26) -> /VIGN
- M1 pad N27: unconnected-(M1-VBAT-PadN27) -> /VBAT
- M1 pad N28: unconnected-(M1-V33_SWITCHABLE-PadN28) -> +3.3VA
- M1 pad N29: unconnected-(M1-OUT_PWR_EN-PadN29) -> /PWR_EN
- M1 pad N30: unconnected-(M1-V5A_SWITCHABLE-PadN30) -> +5VA
- M1 pad N31: unconnected-(M1-VCC-PadN31) -> +5V
- M1 pad N32: unconnected-(M1-V33-PadN32) -> +3.3V
- M1 pad S1: unconnected-(M1-IN_D4-PadS1) -> /D4_IN
- M1 pad S10: unconnected-(M1-IN_AUX4-PadS10) -> /AUX4
- M1 pad S11: unconnected-(M1-IN_AUX3-PadS11) -> /AUX3
- M1 pad S12: unconnected-(M1-IN_AUX2-PadS12) -> /AUX2
- M1 pad S13: unconnected-(M1-IN_AUX1-PadS13) -> /AUX1
- M1 pad S16: unconnected-(M1-IN_O2S-PadS16) -> /O2SENS
- M1 pad S2: unconnected-(M1-IN_D3-PadS2) -> /D3_IN
- M1 pad S23: unconnected-(M1-IN_KNOCK-PadS23) -> /KNOCK_PROCESSED
- M1 pad S25: unconnected-(M1-IN_VSS-PadS25) -> /VSS
- M1 pad S3: unconnected-(M1-IN_D2-PadS3) -> /D2_IN
- M1 pad S35: unconnected-(M1-VREF1-PadS35) -> /VREF1
- M1 pad S4: unconnected-(M1-IN_D1-PadS4) -> /D1_IN
- M1 pad W1: unconnected-(M1-GNDA-PadW1) -> GNDA
- M1 pad W2: unconnected-(M1-V5A_SWITCHABLE-PadW2) -> +5VA
- M2 pad E4: unconnected-(M2-V5_IN-PadE4) -> +5VA
- M2 pad G: unconnected-(M2-GND-PadG) -> GND
- M3 pad E1: unconnected-(M3-Thresh_IN-PadE1) -> /THRESH
- M3 pad E4: unconnected-(M3-V5_IN-PadE4) -> +5VA
- M3 pad G: unconnected-(M3-GND-PadG) -> GND
- M4 pad E1: unconnected-(M4-VBAT-PadE1) -> /VBAT
- M4 pad E3: unconnected-(M4-VIGN-PadE3) -> /VIGN
- M4 pad E4: unconnected-(M4-V5-PadE4) -> +5V
- M4 pad E5: unconnected-(M4-EN_5VP-PadE5) -> /PWR_EN
- M4 pad V4: unconnected-(M4-5VP-PadV4) -> +5VP
Other:
- board outline added: 100 x 100 mm

Commit message: sync
Parts:
- J2: value Conn_02x15_Top_Bottom -> Extra Inputs (2.54mm Pin Header)
- moved U5 61.5 mm to (128.8, 92.0)
- moved U6 61.5 mm to (135.4, 92.0)
- moved M1 48.1 mm to (150.1, 107.3), turned to 0 degrees
- moved M2 17.5 mm to (196.7, 57.9), turned to -90 degrees
- moved M3 17.5 mm to (207.1, 57.9), turned to -90 degrees
- moved U3 11.5 mm to (155.5, 60.0)
- moved M5 5.37 mm to (220.9, 103.2)
- moved J2 4.49 mm to (158.3, 120.5)
- moved U4 1.50 mm to (171.5, 60.0)
Connections:
- J2 pad 1: /LS4_OUT -> /IO1
- J2 pad 10: unconnected-(J2-Pin_10-Pad10) -> /AUX3
- J2 pad 11: unconnected-(J2-Pin_11-Pad11) -> /AUX4
- J2 pad 12: unconnected-(J2-Pin_12-Pad12) -> /D1_IN
- J2 pad 13: unconnected-(J2-Pin_13-Pad13) -> /D2_IN
- J2 pad 14: unconnected-(J2-Pin_14-Pad14) -> /D3_IN
- J2 pad 15: unconnected-(J2-Pin_15-Pad15) -> /D4_IN
- J2 pad 16: unconnected-(J2-Pin_16-Pad16) -> /IO5
- J2 pad 17: unconnected-(J2-Pin_17-Pad17) -> /IO6
- J2 pad 18: unconnected-(J2-Pin_18-Pad18) -> /MAP2
- J2 pad 19: unconnected-(J2-Pin_19-Pad19) -> /MAP3
- J2 pad 2: /LS3_OUT -> /IO2
- J2 pad 20: unconnected-(J2-Pin_20-Pad20) -> /PPS
- J2 pad 21: unconnected-(J2-Pin_21-Pad21) -> /PPS2
- J2 pad 22: unconnected-(J2-Pin_22-Pad22) -> /TPS2
- J2 pad 23: unconnected-(J2-Pin_23-Pad23) -> /AT1
- J2 pad 24: unconnected-(J2-Pin_24-Pad24) -> /AT2
- J2 pad 25: unconnected-(J2-Pin_25-Pad25) -> /O2S2
- J2 pad 26: unconnected-(J2-Pin_26-Pad26) -> /SENS1
- J2 pad 27: unconnected-(J2-Pin_27-Pad27) -> /SENS2
- J2 pad 28: unconnected-(J2-Pin_28-Pad28) -> /SENS3
- J2 pad 29: unconnected-(J2-Pin_29-Pad29) -> /SENS4
- J2 pad 3: /LS2_OUT -> /IO3
- J2 pad 30: unconnected-(J2-Pin_30-Pad30) -> /KNOCK_RAW
- J2 pad 4: /LS1_OUT -> /IO4
- J2 pad 5: /D1_IN -> /RES1
- J2 pad 6: /D2_IN -> /RES2
- J2 pad 7: /D3_IN -> /RES3
- J2 pad 8: /D4_IN -> /AUX1
- J2 pad 9: /KNOCK_RAW -> /AUX2
- M1 pad E1: unconnected-(M1-SPI2_SCK/CAN2_TX-PadE1) -> Net-(M1-SPI2_SCK/CAN2_TX)
- M1 pad E14: /LS3_IN -> unconnected-(M1-OUT_PWM5-PadE14)
- M1 pad E15: /LS2_IN -> unconnected-(M1-OUT_PWM4-PadE15)
- M1 pad E16: /LS1_IN -> unconnected-(M1-OUT_PWM3-PadE16)
- M1 pad E26: /LS4_IN -> unconnected-(M1-OUT_PWM6-PadE26)
- M1 pad E31: unconnected-(M1-OUT_INJ5-PadE31) -> /LS1_IN
- M1 pad E32: unconnected-(M1-OUT_INJ6-PadE32) -> /LS2_IN
- M1 pad E33: unconnected-(M1-OUT_INJ7-PadE33) -> /LS3_IN
- M1 pad E34: unconnected-(M1-OUT_INJ8-PadE34) -> /LS4_IN
- M1 pad E35: unconnected-(M1-IO6-PadE35) -> /IO6
- M1 pad E4: unconnected-(M1-SPI2_CS/CAN2_RX-PadE4) -> Net-(M1-SPI2_CS/CAN2_RX)
- M1 pad N16: unconnected-(M1-IO1-PadN16) -> /IO1
- M1 pad N19: unconnected-(M1-IO2-PadN19) -> /IO2
- M1 pad N20: unconnected-(M1-IO4-PadN20) -> /IO4
- M1 pad N21: unconnected-(M1-IO3-PadN21) -> /IO3
- M1 pad N23: unconnected-(M1-IO5-PadN23) -> /IO5
- M1 pad S14: unconnected-(M1-IN_RES2-PadS14) -> /RES2
- M1 pad S15: unconnected-(M1-IN_O2S2-PadS15) -> /O2S2
- M1 pad S17: unconnected-(M1-IN_RES1-PadS17) -> /RES1
- M1 pad S18: unconnected-(M1-IN_RES3-PadS18) -> /RES3
- M1 pad S19: unconnected-(M1-IN_MAP3-PadS19) -> /MAP3
- M1 pad S20: unconnected-(M1-IN_MAP2-PadS20) -> /MAP2
- M1 pad S27: unconnected-(M1-IN_AT1-PadS27) -> /AT1
- M1 pad S29: unconnected-(M1-IN_AT2-PadS29) -> /AT2
- M1 pad S31: unconnected-(M1-IN_PPS-PadS31) -> /PPS
- M1 pad S32: unconnected-(M1-IN_TPS2-PadS32) -> /TPS2
- M1 pad S33: unconnected-(M1-IN_PPS2-PadS33) -> /PPS2
- M1 pad S6: unconnected-(M1-IN_SENS4-PadS6) -> /SENS4
- M1 pad S7: unconnected-(M1-IN_SENS3-PadS7) -> /SENS3
- M1 pad S8: unconnected-(M1-IN_SENS2-PadS8) -> /SENS2
- M1 pad S9: unconnected-(M1-IN_SENS1-PadS9) -> /SENS1
- M1 pad W12: unconnected-(M1-CANH-PadW12) -> /CAN1+
- M1 pad W13: unconnected-(M1-CANL-PadW13) -> /CAN1-
- M4 pad E6: unconnected-(M4-PG_5VP-PadE6) -> Net-(M4-PG_5VP)
- M5 pad G: unconnected-(M5-GND-PadG) -> GND
- M5 pad W1: unconnected-(M5-V5_IN-PadW1) -> +5VA
- M5 pad W3: unconnected-(M5-CANL-PadW3) -> /CAN1-
- M5 pad W4: unconnected-(M5-CANH-PadW4) -> /CAN1+

Commit message: sync
Parts:
- added J3: TE_6473423-1_26p, TE-6437288-4:64372884, F.Cu at (247.6, 64.1)
- added M7: Module-can-0.1, hellen-one-can:can, F.Cu at (208.0, 115.3)
- added TP1: TestPoint, hellen-one-vr-max9924:vr-max9924, F.Cu at (207.5, 98.7)
- J1: footprint 175446-6:1754466 -> TE-175446-6:1754466
- M1: footprint mega-mcu144:mega-mcu144 -> hellen-one-mega-mcu144:mega-mcu144
- M2: footprint vr-max9924:vr-max9924 -> hellen-one-vr-max9924:vr-max9924
- M3: footprint vr-discrete:vr-discrete -> hellen-one-vr-discrete:vr-discrete
- M4: footprint power_12and5V:power_12and5V -> hellen-one-power_12and5V:power_12and5V
- M5: footprint wbo:wbo -> hellen-one-wbo:wbo
- M6: footprint knock:knock -> hellen-one-knock:knock
- moved M5 60.1 mm to (163.9, 122.2), turned to 0 degrees
- moved M4 55.0 mm to (189.8, 129.0)
- moved M3 29.8 mm to (207.5, 87.7), turned to 0 degrees
- moved M2 21.6 mm to (207.5, 76.6), turned to 0 degrees
- moved J2 19.4 mm to (164.0, 139.0)
- moved M1 1.43 mm to (150.5, 105.9)

Commit message: sync
Parts:
- added BT1: CR1220, kicad6-libraries:CR1220-2, F.Cu at (49.8, 88.2)
- added D10: NUP2105L, Package_TO_SOT_SMD:SOT-23, F.Cu at (207.6, 117.9)
- added F1: Fuse, Fuse:Fuse_1206_3216Metric_Pad1.42x1.75mm_HandSolder, F.Cu at (215.0, 117.7)
- added J5: Conn_01x02, Connector_PinHeader_2.54mm:PinHeader_1x02_P2.54mm_Vertical, F.Cu at (26.0, 109.3)
- added J6: Conn_02x03_Top_Bottom, Connector_Molex:Molex_Mini-Fit_Jr_5566-06A_2x03_P4.20mm_Vertical, F.Cu at (108.0, 120.2)
- added J7: Conn_02x20_Odd_Even, Connector_IDC:IDC-Header_2x20_P2.54mm_Vertical, F.Cu at (138.2, 120.8)
- added J9: Conn_02x06_Top_Bottom, Connector_Molex:Molex_Mini-Fit_Jr_5566-12A_2x06_P4.20mm_Vertical, F.Cu at (206.4, 93.2)
- added L1: 470R@100MHz, Inductor_SMD:L_0603_1608Metric, F.Cu at (203.1, 116.7)
- added L2: 470R@100MHz, Inductor_SMD:L_0603_1608Metric, F.Cu at (203.1, 119.2)
- added U7: MAX31855KASA, Package_SO:SOIC-8_3.9x4.9mm_P1.27mm, F.Cu at (205.3, 112.2)
- added U8: TLE9201SG, Package_SO:Infineon_PG-DSO-12-11, F.Cu at (180.9, 129.5)
- J2: value Extra Inputs (2.54mm Pin Header) -> USB_B; footprint Connector_PinHeader_2.54mm:PinHeader_2x15_P2.54mm_Vertical -> kicad6-libraries:USB_B
- J3: value TE_6473423-1_26p -> Conn_01x02; footprint TE-6437288-4:64372884 -> Connector_PinHeader_2.54mm:PinHeader_1x02_P2.54mm_Vertical
- TP1: footprint hellen-one-vr-max9924:vr-max9924 -> TestPoint:TestPoint_Pad_D1.0mm
- moved M4 170.4 mm to (21.6, 101.7)
- moved TP1 123.4 mm to (87.2, 71.0)
- moved U1 85.9 mm to (197.4, 67.9), turned to 0 degrees
- moved U2 84.3 mm to (197.3, 77.5), turned to 0 degrees
- moved U5 67.2 mm to (196.0, 89.7), turned to 0 degrees
- moved U6 61.2 mm to (196.0, 100.3), turned to 0 degrees
- moved J3 57.6 mm to (214.3, 111.2)
- moved M7 49.5 mm to (163.0, 136.0)
- moved U4 48.0 mm to (123.5, 60.8)
- moved M3 46.0 mm to (169.4, 61.8), turned to -90 degrees
- moved M5 45.9 mm to (118.6, 115.1), turned to 90 degrees
- moved D3 43.1 mm to (67.3, 47.4)
- moved D1 43.1 mm to (67.3, 40.7)
- moved D2 43.1 mm to (67.3, 44.0)
- moved D4 43.1 mm to (67.3, 50.8)
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Connections:
- net /INJ1_IN renamed /LS1_HOT_IN
- net /INJ2_IN renamed /LS2_HOT_IN
- net /INJ3_IN renamed /LS3_HOT_IN
- net /INJ4_IN renamed /LS4_HOT_IN
- J1 pad 106: /SPARK1 -> /5V_OUT1
- J1 pad 112: /INJ1 -> /LS1_HOT_OUT
- J1 pad 125: /INJ2 -> /LS2_HOT_OUT
- J2 pad 1: /IO1 -> Net-(J2-VBUS)
- J2 pad 2: /IO2 -> Net-(J2-D-)
- J2 pad 3: /IO3 -> Net-(J2-D+)
- J2 pad 4: /IO4 -> GND
- J2 pad 5: /RES1 -> GND
- J3 pad 1: unconnected-(J3-Pad1) -> /EGT/T+
- J3 pad 2: unconnected-(J3-Pad2) -> /EGT/T-
- M1 pad E14: unconnected-(M1-OUT_PWM5-PadE14) -> /DC Driver 1/PWM
- M1 pad E35: /IO6 -> unconnected-(M1-IO6-PadE35)
- M1 pad E6: /CHECKCAT_IN -> /DC Driver 1/DIR
- M1 pad E7: unconnected-(M1-OUT_IO5-PadE7) -> /DC Driver 1/DIS
- M1 pad N10: unconnected-(M1-SPI3_CS-PadN10) -> /EGT/SPI_CS
- M1 pad N11: unconnected-(M1-SPI3_SCK-PadN11) -> /EGT/SPI_SCK
- M1 pad N12: unconnected-(M1-SPI3_MISO-PadN12) -> /EGT/SPI_SO
- M1 pad N13: unconnected-(M1-SPI3_MOSI-PadN13) -> /PG
- M1 pad N16: /IO1 -> unconnected-(M1-IO1-PadN16)
- M1 pad N19: /IO2 -> unconnected-(M1-IO2-PadN19)
- M1 pad N2: unconnected-(M1-USBM-PadN2) -> Net-(J2-D-)
- M1 pad N20: /IO4 -> unconnected-(M1-IO4-PadN20)
- M1 pad N21: /IO3 -> unconnected-(M1-IO3-PadN21)
- M1 pad N23: /IO5 -> unconnected-(M1-IO5-PadN23)
- M1 pad N3: unconnected-(M1-USBP-PadN3) -> Net-(J2-D+)
- M1 pad N4: unconnected-(M1-VBUS-PadN4) -> Net-(J2-VBUS)
- M1 pad S14: /RES2 -> unconnected-(M1-IN_RES2-PadS14)
- M1 pad S35: /VREF1 -> unconnected-(M1-VREF1-PadS35)
- M1 pad S5: unconnected-(M1-VREF2-PadS5) -> /VREF1
- M1 pad W10: /SPARK2_OUT -> /5V_OUT2
- M1 pad W11: /SPARK1_OUT -> /5V_OUT1
- M1 pad W12: /CAN1+ -> /CAN2_HIGH
- M1 pad W13: /CAN1- -> /CAN2_LOW
- M1 pad W4: unconnected-(M1-IGN8-PadW4) -> /5V_OUT8
- M1 pad W5: unconnected-(M1-IGN7-PadW5) -> /5V_OUT7
- M1 pad W6: unconnected-(M1-IGN6-PadW6) -> /5V_OUT6
- M1 pad W7: unconnected-(M1-IGN5-PadW7) -> /5V_OUT5
- M1 pad W8: /SPARK4_OUT -> /5V_OUT4
- M1 pad W9: /SPARK3_OUT -> /5V_OUT3
- M4 pad E6: Net-(M4-PG_5VP) -> /PG
- M5 pad W3: /CAN1- -> /CAN1_LOW
- M5 pad W4: /CAN1+ -> /CAN1_HIGH
- M6 pad W1: /KNOCK_RAW -> Net-(J5-Pin_1)
- M7 pad S1: /CAN2- -> /CAN1_LOW
- M7 pad S2: /CAN2+ -> /CAN1_HIGH
- U1 pad 6: /INJ2_OUT -> /LS2_HOT_OUT
- U1 pad 8: /INJ1_OUT -> /LS1_HOT_OUT
- U2 pad 6: /INJ4_OUT -> /LS4_HOT_OUT
- U2 pad 8: /INJ3_OUT -> /LS3_HOT_OUT
Routing:
- added copper zone on B.Cu, net GND
- added copper zone on F.Cu, net GND
- added copper zone on In1.Cu, net GND
- added copper zone on In2.Cu, net GND

Commit message: sync
Parts:
- added C1: 10n, Capacitor_SMD:C_0603_1608Metric, F.Cu at (244.2, 101.5)
- added C10: 10u, Capacitor_SMD:C_0603_1608Metric, F.Cu at (230.2, 111.5)
- added C11: 10u, Capacitor_SMD:C_0603_1608Metric, F.Cu at (234.2, 101.5)
- added C12: 10u, Capacitor_SMD:C_0603_1608Metric, F.Cu at (234.2, 104.0)
- added C13: 10u, Capacitor_SMD:C_0603_1608Metric, F.Cu at (234.2, 106.5)
- added C14: 10u, Capacitor_SMD:C_0603_1608Metric, F.Cu at (234.2, 109.0)
- added C15: 10u, Capacitor_SMD:C_0603_1608Metric, F.Cu at (234.2, 111.5)
- added C16: 100n, Capacitor_SMD:C_0603_1608Metric, F.Cu at (238.2, 101.5)
- added C17: 10n, Capacitor_SMD:C_0603_1608Metric, F.Cu at (238.2, 104.0)
- added C18: 10n, Capacitor_SMD:C_0603_1608Metric, F.Cu at (238.2, 106.5)
- added C2: 100n, Capacitor_SMD:C_0603_1608Metric, F.Cu at (244.2, 104.0)
- added C3: 10n, Capacitor_SMD:C_0603_1608Metric, F.Cu at (244.2, 106.5)
- added C4: 100n, Capacitor_SMD:C_0603_1608Metric, F.Cu at (244.2, 109.0)
- added C5: 1u, Capacitor_SMD:C_0603_1608Metric, F.Cu at (244.2, 111.5)
- added C6: 10u, Capacitor_SMD:C_0603_1608Metric, F.Cu at (230.2, 101.5)
- added C7: 10u, Capacitor_SMD:C_0603_1608Metric, F.Cu at (230.2, 104.0)
- added C8: 10u, Capacitor_SMD:C_0603_1608Metric, F.Cu at (230.2, 106.5)
- added C9: 10u, Capacitor_SMD:C_0603_1608Metric, F.Cu at (230.2, 109.0)
- added R15: 4.7k, Resistor_SMD:R_0603_1608Metric, F.Cu at (238.2, 109.0)
- M1: footprint hellen-one-mega-mcu144:mega-mcu144 -> hellen-one-mega-mcu144-0.7:mega-mcu144
- M2: footprint hellen-one-vr-max9924:vr-max9924 -> hellen-one-vr-max9924-0.3:vr-max9924
- M3: footprint hellen-one-vr-discrete:vr-discrete -> hellen-one-vr-discrete-0.5:vr-discrete
- M5: footprint hellen-one-wbo:wbo -> hellen-one-wbo-0.6:wbo
- M6: footprint hellen-one-knock:knock -> hellen-one-knock-0.2:knock
- M7: footprint hellen-one-can:can -> hellen-one-can-0.1:can
- moved U6 59.5 mm to (242.0, 62.6)
- moved U2 51.4 mm to (242.5, 53.1)
- moved U1 50.8 mm to (242.5, 44.6)
- moved U7 43.6 mm to (239.0, 84.5)
- moved U5 37.8 mm to (228.5, 109.0)
- moved U4 37.2 mm to (160.5, 64.5)
- moved U3 30.7 mm to (150.1, 65.5)
- moved M3 19.3 mm to (188.7, 61.1)
- moved J9 11.7 mm to (203.5, 104.5)
- moved M2 3.21 mm to (176.7, 61.0)
Connections:
- J9 pad 1: /LS4_HOT_OUT -> +12V_RAW
- J9 pad 2: /LS3_HOT_OUT -> GND
- J9 pad 3: /LS2_HOT_OUT -> /LS4_HOT_OUT
- J9 pad 4: /LS1_HOT_OUT -> /LS3_HOT_OUT
- J9 pad 5: +12V_RAW -> /LS2_HOT_OUT
- J9 pad 6: GND -> /LS1_HOT_OUT
Routing:
- net /VR-: track 0.00 -> 14.9 mm
- net /VRCRANK+: track 0.00 -> 10.1 mm
