File: EP91Starlet.kicad_pcb (KiCad board)
At the start: 4 copper layers, 100 x 100 mm, 71 parts, among them J1 175446-6, J2 USB_B, J3 Conn_01x02, J5 Conn_01x02, J6 Conn_02x03_Top_Bottom, J7 Conn_02x20_Odd_Even, J9 Conn_02x06_Top_Bottom, M1 Module-mega-mcu144-0.7, M2 Module-vr-max9924-0.1, M3 Module-vr-discrete-0.5, M4 Module-power_12and5V-0.3, M5 Module-wbo-0.6, M6 Module-knock-0.2, M7 Module-can-0.1, Q2 BSS138, U1 VNLD5090-E, U2 VNLD5090-E, U3 VNLD5090-E, U4 VNLD5090-E, U5 VNLD5090-E, U6 VNLD5090-E, U7 MAX31855KASA, U8 TLE9201SG

Commit message: sync
Parts:
- J6: footprint Connector_Molex:Molex_Mini-Fit_Jr_5566-06A_2x03_P4.20mm_Vertical -> New_Connector_Molex:Molex_Mini-Fit_Jr_5566-06A_2x03_P4.20mm_Vertical
- J9: footprint Connector_Molex:Molex_Mini-Fit_Jr_5566-12A_2x06_P4.20mm_Vertical -> New_Connector_Molex:Molex_Mini-Fit_Jr_5566-12A_2x06_P4.20mm_Vertical
- moved M4 57.9 mm to (79.5, 103.2)
- moved U1 54.4 mm to (192.2, 65.5)
- moved U2 54.4 mm to (192.2, 73.8)
- moved J2 51.4 mm to (196.5, 138.6)
- moved U7 48.1 mm to (212.5, 124.7)
- moved U8 40.8 mm to (203.0, 95.2)
- moved U5 39.7 mm to (212.2, 72.8), turned to 180 degrees
- moved U6 29.9 mm to (212.3, 65.5), turned to 180 degrees
- moved J5 27.4 mm to (52.8, 103.2)
- moved J9 20.8 mm to (199.0, 84.2)
- moved J6 15.2 mm to (122.4, 125.0), turned to -90 degrees
- moved J7 12.9 mm to (147.2, 130.0)
- moved M3 12.7 mm to (176.0, 60.8)
- moved M5 11.8 mm to (126.7, 106.5), turned to -90 degrees
- moved U3 11.5 mm to (138.8, 63.8)
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Connections:
- net /VREF1 renamed /VREF_KNOCK
- J1 pad 106: /5V_OUT1 -> /SPARK
- J1 pad 108: unconnected-(J1-I0F-Pad108) -> /VRCAM+
- J1 pad 112: /LS1_HOT_OUT -> /LS2_HOT_OUT
- J1 pad 125: /LS2_HOT_OUT -> /LS1_HOT_OUT
- J7 pad 1: +5VP -> /D4_IN
- J7 pad 10: /PPS -> +5VP
- J7 pad 11: /AUX4 -> /SENS3
- J7 pad 12: /PPS2 -> +5VP
- J7 pad 13: /AT1 -> /SENS2
- J7 pad 14: /TPS2 -> +5VP
- J7 pad 15: /AT2 -> /SENS1
- J7 pad 16: /O2S2 -> +5VP
- J7 pad 17: /RES1 -> /AUX4
- J7 pad 18: /RES2 -> unconnected-(J7-Pin_18-Pad18)
- J7 pad 19: /D4_IN -> /AUX3
- J7 pad 20: /SENS4 -> unconnected-(J7-Pin_20-Pad20)
- J7 pad 21: /D3_IN -> /AUX2
- J7 pad 22: /SENS3 -> /CAN1+
- J7 pad 23: /D2_IN -> /AUX1
- J7 pad 24: /SENS2 -> /CAN1-
- J7 pad 25: /D1_IN -> /RES2
- J7 pad 26: /SENS1 -> /5V_OUT5
- J7 pad 27: +5VP -> /O2S2
- J7 pad 28: GND -> /5V_OUT4
- J7 pad 29: +5VP -> /MAP3
- J7 pad 3: +5VP -> /D3_IN
- J7 pad 30: GND -> /5V_OUT3
- J7 pad 31: /5V_OUT1 -> /MAP2
- J7 pad 32: /CAN1_HIGH -> /5V_OUT2
- J7 pad 33: /5V_OUT2 -> /AT1
- J7 pad 34: /CAN1_LOW -> /5V_OUT1
- J7 pad 35: /5V_OUT3 -> /AT2
- J7 pad 36: /CAN2_HIGH -> /CAN2-
- J7 pad 37: /5V_OUT4 -> /PPS
- J7 pad 38: /CAN2_LOW -> /CAN2+
- J7 pad 39: unconnected-(J7-Pin_39-Pad39) -> /TPS2
- J7 pad 40: unconnected-(J7-Pin_40-Pad40) -> /PPS2
- J7 pad 5: /AUX1 -> /D2_IN
- J7 pad 6: /MAP2 -> GND
- J7 pad 7: /AUX2 -> /D1_IN
- J7 pad 8: /MAP3 -> GND
- J7 pad 9: /AUX3 -> /SENS4
- J9 pad 10: /LS4_OUT -> /LS2_OUT
- J9 pad 11: /DC1+ -> /LS3_OUT
- J9 pad 12: /DC1- -> /LS4_OUT
- J9 pad 7: /LS1_OUT -> /DC1+
- J9 pad 8: /LS2_OUT -> /DC1-
- J9 pad 9: /LS3_OUT -> /LS1_OUT
- M1 pad E14: /DC Driver 1/PWM -> /THRESH
- M1 pad E28: /THRESH -> /DC Driver 1/PWM
- M1 pad S17: /RES1 -> unconnected-(M1-IN_RES1-PadS17)
- M1 pad S18: /RES3 -> unconnected-(M1-IN_RES3-PadS18)
- M1 pad W10: /5V_OUT2 -> /5V_OUT1
- M1 pad W11: /5V_OUT1 -> /SPARK
- M1 pad W12: /CAN2_HIGH -> /CAN2+
- M1 pad W13: /CAN2_LOW -> /CAN2-
- M1 pad W4: /5V_OUT8 -> /5V_OUT7
- M1 pad W5: /5V_OUT7 -> /5V_OUT6
- M1 pad W6: /5V_OUT6 -> /5V_OUT5
- M1 pad W7: /5V_OUT5 -> /5V_OUT4
- M1 pad W8: /5V_OUT4 -> /5V_OUT3
- M1 pad W9: /5V_OUT3 -> /5V_OUT2
- M3 pad W2: unconnected-(M3-VR+-PadW2) -> /VRCAM+
- M5 pad W3: /CAN1_LOW -> /CAN1-
- M5 pad W4: /CAN1_HIGH -> /CAN1+
- M7 pad S1: /CAN1_LOW -> /CAN1-
- M7 pad S2: /CAN1_HIGH -> /CAN1+
Routing:
- net /THRESH: track 0.00 -> 72.7 mm
- net /5V_OUT1: track 0.00 -> 58.3 mm
- net /VSS: track 0.00 -> 58.1 mm, vias 0 -> 1
- net /CAM: track 0.00 -> 57.1 mm, vias 0 -> 2
- net /CAN2-: track 0.00 -> 54.8 mm
- net /5V_OUT2: track 0.00 -> 53.7 mm
- net /CAN2+: track 0.00 -> 52.3 mm
- net /CRANK: track 0.00 -> 49.2 mm, vias 0 -> 2
- net /5V_OUT3: track 0.00 -> 49.2 mm
- net /MAP: track 0.00 -> 47.3 mm
- net /TPS: track 0.00 -> 44.7 mm
- net /5V_OUT4: track 0.00 -> 44.6 mm
- net /AIR: track 0.00 -> 41.9 mm
- net /COOLANT: track 0.00 -> 40.2 mm, vias 0 -> 1
- net /5V_OUT5: track 0.00 -> 40.0 mm
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
Commit message: sync
Parts:
- moved M4 121.7 mm to (195.6, 66.8)
- moved J2 107.0 mm to (89.5, 138.6)
- moved U1 71.6 mm to (196.5, 137.0)
- moved U2 69.6 mm to (190.5, 143.4)
- moved U5 69.6 mm to (210.7, 142.4)
- moved U6 69.6 mm to (210.8, 135.1)
- moved J9 63.9 mm to (160.3, 135.0), turned to 0 degrees
- moved Q2 46.2 mm to (127.5, 61.9), turned to 90 degrees
- moved M7 46.1 mm to (207.9, 137.9)
- moved U8 40.3 mm to (196.8, 135.0), turned to 180 degrees
- moved J6 8.25 mm to (124.6, 133.0), turned to 0 degrees
- moved M5 5.52 mm to (122.6, 102.8)
- moved U4 0.79 mm to (152.0, 64.0)
- moved U3 0.25 mm to (138.8, 64.0)
Connections:
- J6 pad 1: unconnected-(J6-Pin_1-Pad1) -> Net-(J6-Pin_1)
- J6 pad 2: unconnected-(J6-Pin_2-Pad2) -> Net-(J6-Pin_2)
- J6 pad 3: unconnected-(J6-Pin_3-Pad3) -> Net-(J6-Pin_3)
- J6 pad 4: unconnected-(J6-Pin_4-Pad4) -> Net-(J6-Pin_4)
- J6 pad 5: unconnected-(J6-Pin_5-Pad5) -> +12V_RAW
- J6 pad 6: unconnected-(J6-Pin_6-Pad6) -> Net-(J6-Pin_6)
- M5 pad E1: unconnected-(M5-LSU_Un-PadE1) -> Net-(J6-Pin_4)
- M5 pad E2: unconnected-(M5-LSU_Vm-PadE2) -> Net-(J6-Pin_6)
- M5 pad E3: unconnected-(M5-LSU_Ip-PadE3) -> Net-(J6-Pin_3)
- M5 pad E4: unconnected-(M5-LSU_Rtrim-PadE4) -> Net-(J6-Pin_1)
- M5 pad E5: unconnected-(M5-LSU_Htr-PadE5) -> Net-(J6-Pin_2)
Routing:
- net +12V_RAW: track 0.00 -> 80.6 mm
- net +12V_PERM: track 0.00 -> 75.7 mm
- net /VBAT: track 0.00 -> 64.5 mm, vias 0 -> 1
- net /VIGN: track 0.00 -> 55.2 mm
- net +5V: track 0.00 -> 41.5 mm
- net +5VP: track 0.00 -> 39.8 mm
- net /VSS: track 58.1 -> 55.7 mm

Commit message: sync
Parts:
- BT1: moved to B.Cu
- moved J2 138.2 mm to (227.7, 141.8)
- moved M7 74.0 mm to (137.5, 115.2), turned to 180 degrees
- moved M6 73.6 mm to (126.6, 132.8)
- moved J6 62.8 mm to (127.2, 70.3), turned to -90 degrees
- moved BT1 43.5 mm to (82.5, 116.9), turned to 180 degrees
- moved M5 16.3 mm to (138.4, 106.9), turned to 90 degrees
- moved J9 6.49 mm to (163.9, 140.4)
Connections:
- J7 pad 18: unconnected-(J7-Pin_18-Pad18) -> /CAN1-
- J7 pad 20: unconnected-(J7-Pin_20-Pad20) -> /CAN1+
- J7 pad 22: /CAN1+ -> unconnected-(J7-Pin_22-Pad22)
- J7 pad 24: /CAN1- -> unconnected-(J7-Pin_24-Pad24)
Routing:
- net Net-(M1-SPI2_SCK/CAN2_TX): track 0.00 -> 66.3 mm
- net Net-(M1-SPI2_CS/CAN2_RX): track 0.00 -> 63.2 mm
- net +12V_RAW: track 80.6 -> 104.8 mm
- net Net-(J6-Pin_4): track 0.00 -> 21.2 mm
- net Net-(J6-Pin_1): track 0.00 -> 16.0 mm
- net Net-(J6-Pin_6): track 0.00 -> 14.4 mm
- net /CAN1+: track 0.00 -> 13.4 mm
- net /CAN1-: track 0.00 -> 12.6 mm
- net Net-(J6-Pin_2): track 0.00 -> 11.0 mm
- net Net-(J6-Pin_3): track 0.00 -> 9.69 mm
