File: EP91Starlet.kicad_pcb (KiCad board)
At the start: 4 copper layers, 100 x 100 mm, 74 parts, among them IC1 VNLD5160-E, IC2 VNLD5160-E, IC3 VNLD5160-E, IC4 VNLD5160-E, IC5 VNLD5160-E, IC6 VNLD5160-E, J1 175446-6, J3 Conn_01x02, J4 USB_B_Mini, J5 Conn_01x02, J6 Conn_02x03_Top_Bottom, J7 Conn_02x20_Odd_Even, J9 Conn_02x06_Top_Bottom, M1 Module-mega-mcu144-0.7, M2 Module-vr-max9924-0.1, M3 Module-vr-discrete-0.5, M4 Module-power_12and5V-0.3, M5 Module-wbo-0.6, M6 Module-knock-0.2, M7 Module-can-0.1, Q2 BSS138, U7 MAX31855KASA, U8 TLE9201SG

Commit message: sync
Parts:
- Q2, R10, R9: moved to B.Cu
- moved Q2 120.5 mm to (128.4, 34.2), turned to -90 degrees
- moved R9 55.5 mm to (128.6, 26.9), turned to 180 degrees
- moved R10 53.6 mm to (128.6, 31.4), turned to 180 degrees
- moved U7 23.7 mm to (193.8, 90.8)
- moved J4 17.5 mm to (156.8, 125.4)
- moved D10 15.1 mm to (97.3, 39.5)
- moved J5 13.3 mm to (82.2, 83.9), turned to 180 degrees
- moved M7 11.1 mm to (166.3, 127.6)
- moved D2 11.0 mm to (139.2, 34.7)
- moved D1 11.0 mm to (139.2, 31.4)
- moved IC1 9.66 mm to (216.7, 63.2)
- moved J3 9.62 mm to (203.1, 89.6)
- moved M6 5.83 mm to (92.0, 79.2)
- moved J9 1.30 mm to (200.3, 65.8)
- moved IC3 1.24 mm to (152.3, 34.2)
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Connections:
- net Net-(J4-D-) renamed /USB-
- J4 pad 1: /USB+ -> Net-(J4-VBUS)
- J4 pad 3: Net-(J4-D+) -> /USB+
- M1 pad E12: /CHECKENGINE_IN -> unconnected-(M1-OUT_IO2-PadE12)
- M1 pad E13: unconnected-(M1-OUT_IO12-PadE13) -> /DC Driver 1/DIR
- M1 pad E15: unconnected-(M1-OUT_PWM4-PadE15) -> /IACOPEN_IN
- M1 pad E16: unconnected-(M1-OUT_PWM3-PadE16) -> /IACCLOSE_IN
- M1 pad E17: /IACOPEN_IN -> unconnected-(M1-OUT_PWM2-PadE17)
- M1 pad E20: unconnected-(M1-OUT_IO13-PadE20) -> /DC Driver 1/DIS
- M1 pad E21: /FANRELAY_IN -> unconnected-(M1-OUT_IO4-PadE21)
- M1 pad E26: unconnected-(M1-OUT_PWM6-PadE26) -> /DC Driver 1/PWM
- M1 pad E27: /IACCLOSE_IN -> unconnected-(M1-OUT_PWM1-PadE27)
- M1 pad E28: /DC Driver 1/PWM -> unconnected-(M1-OUT_PWM8-PadE28)
- M1 pad E6: /DC Driver 1/DIR -> /FANRELAY_IN
- M1 pad E7: /DC Driver 1/DIS -> /FUELRELAY_IN
- M1 pad E8: /FUELRELAY_IN -> /CHECKENGINE_IN
- M1 pad N3: Net-(J4-D+) -> /USB+
- M1 pad N4: /USB+ -> Net-(J4-VBUS)
Routing:
- net /THRESH: track 0.00 -> 67.3 mm, vias 0 -> 1
- net /IACCLOSE_IN: track 0.00 -> 29.6 mm, vias 0 -> 1
- net /IACOPEN_IN: track 0.00 -> 28.2 mm, vias 0 -> 1
- net /CHECKENGINE_IN: track 0.00 -> 21.7 mm, vias 0 -> 1
- net /FUELRELAY_IN: track 0.00 -> 20.6 mm, vias 0 -> 1
- net /FANRELAY_IN: track 0.00 -> 20.3 mm, vias 0 -> 1
- net /CRANK: track 70.4 -> 69.1 mm
- net /TPS: track 58.5 -> 57.5 mm
- net /MAP: track 66.0 -> 65.0 mm
- net /CAM: track 56.9 -> 56.3 mm
